Commit message: reemc_description: revert hardware_interfaces in joints

File: reemc_description/urdf/arm/arm.transmission.xacro (robot description, xacro)
@@ -13,7 +13,8 @@
       <actuator name="${name}_${side}_${number}_motor" >
         <mechanicalReduction>${reduction}</mechanicalReduction>
+      </actuator>
+      <joint name="${name}_${side}_${number}_joint">
         <hardwareInterface>hardware_interface/PositionJointInterface</hardwareInterface>
-      </actuator>
-      <joint name="${name}_${side}_${number}_joint" />
+      </joint>
     </transmission>
   </xacro:macro>

File: reemc_description/urdf/arm/wrist.transmission.xacro (robot description, xacro)
@@ -13,7 +13,8 @@
       <actuator name="${name}_${side}_${number}_motor" >
         <mechanicalReduction>${reduction}</mechanicalReduction>
+      </actuator>
+      <joint name="${name}_${side}_${number}_joint">
         <hardwareInterface>hardware_interface/PositionJointInterface</hardwareInterface>
-      </actuator>
-      <joint name="${name}_${side}_${number}_joint" />
+      </joint>
     </transmission>
   </xacro:macro>
@@ -25,10 +26,8 @@
         <role>actuator1</role>
         <mechanicalReduction>${act_reduction_1}</mechanicalReduction>
-        <hardwareInterface>hardware_interface/PositionJointInterface</hardwareInterface>
       </actuator>
       <actuator name="${name}_${side}_${number_2}_motor">
         <role>actuator2</role>
         <mechanicalReduction>${act_reduction_2}</mechanicalReduction>
-        <hardwareInterface>hardware_interface/PositionJointInterface</hardwareInterface>
       </actuator>
       <joint name="${name}_${side}_${number_1}_joint">
@@ -36,4 +35,5 @@
         <offset>0.0</offset>
         <mechanicalReduction>${jnt_reduction_1}</mechanicalReduction>
+        <hardwareInterface>hardware_interface/PositionJointInterface</hardwareInterface>
       </joint>
       <joint name="${name}_${side}_${number_2}_joint">
@@ -41,4 +41,5 @@
         <offset>0.0</offset>
         <mechanicalReduction>${jnt_reduction_2}</mechanicalReduction>
+        <hardwareInterface>hardware_interface/PositionJointInterface</hardwareInterface>
       </joint>
     </transmission>

File: reemc_description/urdf/hand/hand.transmission.xacro (robot description, xacro)
@@ -14,7 +14,8 @@
       <actuator name="${name}_motor" >
         <mechanicalReduction>${reduction}</mechanicalReduction>
+      </actuator>
+      <joint name="${name}_joint" >
         <hardwareInterface>hardware_interface/PositionJointInterface</hardwareInterface>
-      </actuator>
-      <joint name="${name}_joint" />
+      </joint>
     </transmission>
   </xacro:macro>
@@ -27,7 +28,8 @@
       <actuator name="${finger_name}_motor" >
         <mechanicalReduction>${actuator_reduction}</mechanicalReduction>
+      </actuator>
+      <joint name="${finger_name}_joint" >
         <hardwareInterface>hardware_interface/PositionJointInterface</hardwareInterface>
-      </actuator>
-      <joint name="${finger_name}_joint" />
+      </joint>
     </transmission>
     <!-- Read-only finger phalanxes -->
@@ -36,7 +38,8 @@
       <actuator name="${finger_name}_1_motor" >
         <mechanicalReduction>1.0</mechanicalReduction>
+      </actuator>
+      <joint name="${finger_name}_1_joint" >
         <hardwareInterface>hardware_interface/JointStateInterface</hardwareInterface>
-      </actuator>
-      <joint name="${finger_name}_1_joint" />
+      </joint>
     </transmission>
     <transmission name="${finger_name}_2_trans">
@@ -44,7 +47,8 @@
       <actuator name="${finger_name}_2_motor" >
         <mechanicalReduction>1.0</mechanicalReduction>
+      </actuator>
+      <joint name="${finger_name}_2_joint" >
         <hardwareInterface>hardware_interface/JointStateInterface</hardwareInterface>
-      </actuator>
-      <joint name="${finger_name}_2_joint" />
+      </joint>
     </transmission>
     <transmission name="${finger_name}_3_trans">
@@ -52,7 +56,8 @@
       <actuator name="${finger_name}_3_motor" >
         <mechanicalReduction>1.0</mechanicalReduction>
+      </actuator>
+      <joint name="${finger_name}_3_joint" >
         <hardwareInterface>hardware_interface/JointStateInterface</hardwareInterface>
-      </actuator>
-      <joint name="${finger_name}_3_joint" />
+      </joint>
     </transmission>
   </xacro:macro>

File: reemc_description/urdf/head/head.transmission.xacro (robot description, xacro)
@@ -13,7 +13,8 @@
       <actuator name="${name}_motor" >
         <mechanicalReduction>${reduction}</mechanicalReduction>
+      </actuator>
+      <joint name="${name}_joint" >
         <hardwareInterface>hardware_interface/PositionJointInterface</hardwareInterface>
-      </actuator>
-      <joint name="${name}_joint" />
+      </joint>
     </transmission>
   </xacro:macro>

File: reemc_description/urdf/leg/leg.transmission.xacro (robot description, xacro)
@@ -13,7 +13,8 @@
       <actuator name="${name}_${side}_${number}_motor" >
         <mechanicalReduction>${reduction}</mechanicalReduction>
+      </actuator>
+      <joint name="${name}_${side}_${number}_joint">
         <hardwareInterface>hardware_interface/PositionJointInterface</hardwareInterface>
-      </actuator>
-      <joint name="${name}_${side}_${number}_joint" />
+      </joint>
     </transmission>
   </xacro:macro>

File: reemc_description/urdf/torso/torso.transmission.xacro (robot description, xacro)
@@ -15,10 +15,8 @@
         <role>actuator1</role>
         <mechanicalReduction>${act_reduction1}</mechanicalReduction>
-        <hardwareInterface>hardware_interface/PositionJointInterface</hardwareInterface>
       </actuator>
       <actuator name="${name}_${number2}_motor">
         <role>actuator2</role>
         <mechanicalReduction>${act_reduction2}</mechanicalReduction>
-        <hardwareInterface>hardware_interface/PositionJointInterface</hardwareInterface>
       </actuator>
       <joint name="${name}_${number1}_joint">
@@ -26,4 +24,5 @@
         <offset>0.0</offset>
         <mechanicalReduction>${jnt_reduction1}</mechanicalReduction>
+        <hardwareInterface>hardware_interface/PositionJointInterface</hardwareInterface>
       </joint>
       <joint name="${name}_${number2}_joint">
@@ -31,4 +30,5 @@
         <offset>0.0</offset>
         <mechanicalReduction>${jnt_reduction2}</mechanicalReduction>
+        <hardwareInterface>hardware_interface/PositionJointInterface</hardwareInterface>
       </joint>
     </transmission>
