Commit message: Changed cfmDamping instances for implicitSpringDamper instances. The first one was deprecated, so we get rid of all the deprecated warnings
git-svn-id: svn+ssh://server/srv/svn/repos/trunk/pal-ros-pkg/catkin_pkgs/reemc_robot@52256 5e370ff8-3418-0410-babe-3378cc20a00d

File: reemc_description/urdf/arm/arm.urdf.xacro (robot description, xacro)
@@ -188,14 +188,14 @@
    </gazebo>
    <gazebo reference="${name}_${side}_1_joint">
-      <cfmDamping>1</cfmDamping>
+      <implicitSpringDamper>1</implicitSpringDamper>
    </gazebo>
    <gazebo reference="${name}_${side}_2_joint">
-      <cfmDamping>1</cfmDamping>
+      <implicitSpringDamper>1</implicitSpringDamper>
    </gazebo>
    <gazebo reference="${name}_${side}_3_joint">
-      <cfmDamping>1</cfmDamping>
+      <implicitSpringDamper>1</implicitSpringDamper>
    </gazebo>
    <gazebo reference="${name}_${side}_4_joint">
-      <cfmDamping>1</cfmDamping>
+      <implicitSpringDamper>1</implicitSpringDamper>
    </gazebo>
     <!--************************-->

File: reemc_description/urdf/arm/wrist.urdf.xacro (robot description, xacro)
@@ -141,11 +141,11 @@
     </gazebo>
     <gazebo reference="${name}_${side}_5_joint">
-        <cfmDamping>1</cfmDamping>
+        <implicitSpringDamper>1</implicitSpringDamper>
     </gazebo>
     <gazebo reference="${name}_${side}_6_joint">
-        <cfmDamping>1</cfmDamping>
+        <implicitSpringDamper>1</implicitSpringDamper>
     </gazebo>
     <gazebo reference="${name}_${side}_7_joint">
-        <cfmDamping>1</cfmDamping>
+        <implicitSpringDamper>1</implicitSpringDamper>
     </gazebo>
     <!-- extensions -->

File: reemc_description/urdf/foot/foot.urdf.xacro (robot description, xacro)
@@ -22,5 +22,5 @@
     </visual>
     <!-- bottom -->
-    <collision group="default">
+    <collision>
       <origin rpy="0 0 0" xyz="0.048 0 -0.076119"/>
       <geometry>

File: reemc_description/urdf/hand/hand.gazebo.xacro (robot description, xacro)
@@ -60,17 +60,17 @@
     </gazebo>
     <gazebo reference="${finger_name}_joint">
-      <cfmDamping>1</cfmDamping>
+      <implicitSpringDamper>1</implicitSpringDamper>
       <provideFeedback>1</provideFeedback>
     </gazebo>
     <gazebo reference="${finger_name}_1_joint">
-      <cfmDamping>1</cfmDamping>
+      <implicitSpringDamper>1</implicitSpringDamper>
       <provideFeedback>1</provideFeedback>
     </gazebo>
     <gazebo reference="${finger_name}_2_joint">
-      <cfmDamping>1</cfmDamping>
+      <implicitSpringDamper>1</implicitSpringDamper>
       <provideFeedback>1</provideFeedback>
     </gazebo>
     <gazebo reference="${finger_name}_3_joint">
-      <cfmDamping>1</cfmDamping>
+      <implicitSpringDamper>1</implicitSpringDamper>
       <provideFeedback>1</provideFeedback>
     </gazebo>

File: reemc_description/urdf/hand/hand.urdf.xacro (robot description, xacro)
@@ -222,5 +222,5 @@
     </gazebo>
     <gazebo reference="${name}_${side}_thumb_joint">
-       <cfmDamping>1</cfmDamping>
+       <implicitSpringDamper>1</implicitSpringDamper>
     </gazebo>
     <!-- Grasping frame -->

File: reemc_description/urdf/head/head.urdf.xacro (robot description, xacro)
@@ -60,5 +60,5 @@
     </gazebo>
     <gazebo reference="${name}_joint">
-       <cfmDamping>1</cfmDamping>
+       <implicitSpringDamper>1</implicitSpringDamper>
     </gazebo>
     <!-- extensions -->
@@ -109,5 +109,5 @@
     </gazebo>
     <gazebo reference="${name}_joint">
-       <cfmDamping>1</cfmDamping>
+       <implicitSpringDamper>1</implicitSpringDamper>
     </gazebo>
     <!-- Head Sonar -->

File: reemc_description/urdf/leg/leg.urdf.xacro (robot description, xacro)
@@ -96,5 +96,5 @@
         <material name="LightGrey" />
       </visual>
-      <collision group="default">
+      <collision>
         <origin rpy="0 ${90* deg_to_rad} 0" xyz="0.15 0 ${-reflect*0.015}"/>
         <geometry>
@@ -128,5 +128,5 @@
         <material name="LightGrey" />
       </visual>
-      <collision group="default">
+      <collision>
         <origin rpy="0 ${-reflect* 90* deg_to_rad} 0" xyz="0.15 0 ${-reflect*0.015}"/>
         <geometry>
@@ -251,25 +251,25 @@
      <maxVel>1.0</maxVel>
      <minDepth>0.00</minDepth>
-     <cfmDamping>1</cfmDamping>
+     <implicitSpringDamper>1</implicitSpringDamper>
    </gazebo>
    <!--force torque sensor -->
    <!--xacro:reemc_force_torque_sensor name="leg_${side}_6_link"  update_rate="100.0"/-->
    <gazebo reference="leg_${side}_1_joint">
-      <cfmDamping>1</cfmDamping>
+      <implicitSpringDamper>1</implicitSpringDamper>
    </gazebo>
    <gazebo reference="leg_${side}_2_joint">
-      <cfmDamping>1</cfmDamping>
+      <implicitSpringDamper>1</implicitSpringDamper>
    </gazebo>
    <gazebo reference="leg_${side}_3_joint">
-      <cfmDamping>1</cfmDamping>
+      <implicitSpringDamper>1</implicitSpringDamper>
    </gazebo>
    <gazebo reference="leg_${side}_4_joint">
-      <cfmDamping>1</cfmDamping>
+      <implicitSpringDamper>1</implicitSpringDamper>
    </gazebo>
    <gazebo reference="leg_${side}_5_joint">
-      <cfmDamping>1</cfmDamping>
+      <implicitSpringDamper>1</implicitSpringDamper>
    </gazebo>
    <gazebo reference="leg_${side}_6_joint">
-     <cfmDamping>1</cfmDamping>
+     <implicitSpringDamper>1</implicitSpringDamper>
      <provideFeedback>1</provideFeedback>
    </gazebo>

File: reemc_description/urdf/torso/torso.urdf.xacro (robot description, xacro)
@@ -91,8 +91,8 @@
    </gazebo>
    <gazebo reference="${name}_1_joint">
-      <cfmDamping>1</cfmDamping>
+      <implicitSpringDamper>1</implicitSpringDamper>
    </gazebo>
    <gazebo reference="${name}_2_joint">
-     <cfmDamping>1</cfmDamping>
+     <implicitSpringDamper>1</implicitSpringDamper>
      <provideFeedback>1</provideFeedback>
    </gazebo>
