Commit message: reemc_description: remove unused force_torque sensor plugin

File: reemc_description/urdf/sensors/ftsensor.gazebo.xacro (robot description, xacro)
@@ -17,15 +17,9 @@
          <collision>${name}_collision</collision>
        </contact>
-       <plugin filename="libgazebo_ros_forcetorque.so" name="${name}_ft_plugin">
-         <robotNamespace></robotNamespace>
-         <topicName>${name}_ft_data</topicName>
-         <frameName>${name}</frameName>
-         <updateRate>${update_rate}</updateRate>
-       </plugin>
-     </sensor>
-   </gazebo>
-   <gazebo reference="${name}">
-     <provideFeedback>1</provideFeedback>
-   </gazebo>
- </xacro:macro>
+   </sensor>
+</gazebo>
+<gazebo reference="${name}">
+  <provideFeedback>1</provideFeedback>
+</gazebo>
+</xacro:macro>
 </robot>

Commit message: reemc_description: ftplugin not needed anymore
git-svn-id: svn+ssh://server/srv/svn/repos/branches/hydro_migration/pal-ros-pkg/catkin_pkgs/reemc_robot@48958 5e370ff8-3418-0410-babe-3378cc20a00d

File: reemc_description/urdf/sensors/ftsensor.gazebo.xacro (robot description, xacro)
@@ -12,20 +12,14 @@
     <sensor name="${name}_contact_sensor" type="contact">
       <pose>0.105 0.071 0 0 0 0</pose>
-       <always_on>1</always_on>
-       <update_rate>${update_rate}</update_rate>
-       <contact>
-         <collision>${name}_collision</collision>
-       </contact>
-       <plugin filename="libgazebo_ros_forcetorque.so" name="${name}_ft_plugin">
-         <robotNamespace></robotNamespace>
-         <topicName>${name}_ft_data</topicName>
-         <frameName>${name}</frameName>
-         <updateRate>${update_rate}</updateRate>
-       </plugin>
-     </sensor>
-   </gazebo>
-   <gazebo reference="${name}">
-     <provideFeedback>1</provideFeedback>
-   </gazebo>
- </xacro:macro>
+      <always_on>1</always_on>
+      <update_rate>${update_rate}</update_rate>
+      <contact>
+        <collision>${name}_collision</collision>
+      </contact>
+    </sensor>
+  </gazebo>
+  <gazebo reference="${name}">
+    <provideFeedback>1</provideFeedback>
+  </gazebo>
+</xacro:macro>
 </robot>
