Commit message: Added nice spacewq

File: reemc_description/urdf/sensors/ftsensor.urdf.xacro (robot description, xacro)
@@ -8,8 +8,8 @@
 -->
 <robot xmlns:xacro="http://ros.org/wiki/xacro">
- <xacro:macro name="ft_sensor" params="name parent side reflect">
- <!--************************-->
- <!--        ft sensor        -->
- <!--************************-->
+  <xacro:macro name="ft_sensor" params="name parent side reflect">
+    <!--************************-->
+    <!--        ft sensor       -->
+    <!--************************-->
     <link name="${name}_${side}_ft_link">
       <inertial>
@@ -37,5 +37,5 @@
     </joint>
     <!--***********************-->
-    <!--       FT TOOL           -->
+    <!--       FT TOOL         -->
     <!--***********************-->
     <link name="${name}_${side}_ft_tool_link">
