Commit message: Use pi instead of M_PI

File: reemc_description/urdf/sensors/back_camera.urdf.xacro (robot description, xacro)
@@ -40,5 +40,5 @@
     <!-- attach optical frame to the camera link -->
     <joint name="${name}_optical_frame_joint" type="fixed">
-      <origin xyz="0 0 0" rpy="${-M_PI/2} 0.0 ${-M_PI/2}" /> <!-- rotate frame from x-forward to z-forward camera coords -->
+      <origin xyz="0 0 0" rpy="${-pi/2} 0.0 ${-pi/2}" /> <!-- rotate frame from x-forward to z-forward camera coords -->
       <parent link="${name}_link"/>
       <child link="${name}_optical_frame"/>

File: reemc_description/urdf/sensors/stereo_camera.urdf.xacro (robot description, xacro)
@@ -48,5 +48,5 @@
     <!-- attach optical frame to the camera link -->
     <joint name="${name}_optical_frame_joint" type="fixed">
-      <origin xyz="0 0 0" rpy="${-M_PI/2} 0.0 ${-M_PI/2}" /> <!-- rotate frame from x-forward to z-forward camera coords -->
+      <origin xyz="0 0 0" rpy="${-pi/1} 0.0 ${-pi/2}" /> <!-- rotate frame from x-forward to z-forward camera coords -->
       <parent link="${name}_link"/>
       <child link="${name}_optical_frame"/>
