Commit message: Spread change from REEM-H model: Changed the multiplier of the mimic joints of the finger so the movement of the active joint spreads corretly to the subactuated joints
git-svn-id: svn+ssh://server/srv/svn/repos/trunk/pal-ros-pkg/catkin_pkgs/reemc_robot@52205 5e370ff8-3418-0410-babe-3378cc20a00d

File: reemc_description/urdf/hand/hand.urdf.xacro (robot description, xacro)
@@ -9,7 +9,7 @@
 <robot xmlns:xacro="http://ros.org/wiki/xacro">
   <!--File includes-->
-  <xacro:include filename="$(find reemc_description)/urdf/deg_to_rad.xacro" />
-  <xacro:include filename="$(find reemc_description)/urdf/hand/hand.gazebo.xacro" />
-  <xacro:include filename="$(find reemc_description)/urdf/hand/hand.transmission.xacro" />
+  <xacro:include filename="$(find reem_description)/urdf/deg_to_rad.xacro" />
+  <xacro:include filename="$(find reem_description)/urdf/hand/hand.gazebo.xacro" />
+  <xacro:include filename="$(find reem_description)/urdf/hand/hand.transmission.xacro" />
   <!--Constant parameters-->
   <xacro:property name="hand_friction" value="0.0" /> <!--TODO: Tune-->
@@ -59,5 +59,5 @@
       <limit lower="${0.0 * deg_to_rad}" upper="${90.0 * deg_to_rad}" effort="2.0" velocity="${hand_max_vel}" />
       <dynamics friction="${hand_friction}" damping="${hand_damping}"/>
-      <mimic joint="${hand_name}_${hand_side}_${finger_name}_joint" multiplier="-1.0" offset="0.0" />
+      <mimic joint="${hand_name}_${hand_side}_${finger_name}_joint" multiplier="${90.0 / 250.0}" offset="0.0" />
     </joint>
     <link name="${hand_name}_${hand_side}_${finger_name}_1_link">
@@ -70,12 +70,12 @@
         <origin xyz="0 0 0" rpy="0 0 0" />
         <geometry>
-          <mesh filename="package://reemc_description/meshes/hand/hand_finger_1.dae" scale="1 1 ${-reflect * finger_reflect * 1}" />
-        </geometry>
-        <material name="LightGrey" />
-      </visual>
-      <collision>
-        <origin xyz="0 0 0" rpy="0 0 0" />
-        <geometry>
-          <mesh filename="package://reemc_description/meshes/hand/hand_finger_1_collision.stl" scale="1 1 ${-reflect * finger_reflect}" />
+          <mesh filename="package://reem_description/meshes/hand/hand_finger_1.dae" scale="1 1 ${-reflect * finger_reflect * 1}" />
+        </geometry>
+        <material name="LightGrey" />
+      </visual>
+      <collision>
+        <origin xyz="0 0 0" rpy="0 0 0" />
+        <geometry>
+          <mesh filename="package://reem_description/meshes/hand/hand_finger_1_collision.stl" scale="1 1 ${-reflect * finger_reflect}" />
         </geometry>
       </collision>
@@ -88,5 +88,5 @@
       <limit lower="${0.0 * deg_to_rad}" upper="${80.0 * deg_to_rad}" effort="1.0" velocity="${hand_max_vel}" />
       <dynamics friction="${hand_friction}" damping="${hand_damping}"/>
-      <mimic joint="${hand_name}_${hand_side}_${finger_name}_joint" multiplier="-1.0" offset="0.0" />
+      <mimic joint="${hand_name}_${hand_side}_${finger_name}_joint" multiplier="${80.0 / 250.0}" offset="0.0" />
     </joint>
     <link name="${hand_name}_${hand_side}_${finger_name}_2_link">
@@ -99,12 +99,12 @@
         <origin xyz="0 0 0" rpy="0 0 0" />
         <geometry>
-          <mesh filename="package://reemc_description/meshes/hand/hand_finger_2.dae" scale="1 1 ${-reflect * finger_reflect * 1}" />
-        </geometry>
-        <material name="LightGrey" />
-      </visual>
-      <collision>
-        <origin xyz="0 0 0" rpy="0 0 0" />
-        <geometry>
-          <mesh filename="package://reemc_description/meshes/hand/hand_finger_2_collision.stl" scale="1 1 ${-reflect * finger_reflect}" />
+          <mesh filename="package://reem_description/meshes/hand/hand_finger_2.dae" scale="1 1 ${-reflect * finger_reflect * 1}" />
+        </geometry>
+        <material name="LightGrey" />
+      </visual>
+      <collision>
+        <origin xyz="0 0 0" rpy="0 0 0" />
+        <geometry>
+          <mesh filename="package://reem_description/meshes/hand/hand_finger_2_collision.stl" scale="1 1 ${-reflect * finger_reflect}" />
         </geometry>
       </collision>
@@ -117,5 +117,5 @@
       <limit lower="${0.0 * deg_to_rad}" upper="${80.0 * deg_to_rad}" effort="1.0" velocity="${hand_max_vel}" />
       <dynamics friction="${hand_friction}" damping="${hand_damping}"/>
-      <mimic joint="${hand_name}_${hand_side}_${finger_name}_joint" multiplier="-1.0" offset="0.0" />
+      <mimic joint="${hand_name}_${hand_side}_${finger_name}_joint" multiplier="${80.0 / 250.0}" offset="0.0" />
     </joint>
     <link name="${hand_name}_${hand_side}_${finger_name}_3_link">
@@ -128,12 +128,12 @@
         <origin xyz="0 0 0" rpy="0 0 0" />
         <geometry>
-          <mesh filename="package://reemc_description/meshes/hand/hand_finger_3.dae" scale="1 1 ${-reflect * finger_reflect*1}" />
-        </geometry>
-        <material name="LightGrey" />
-      </visual>
-      <collision>
-        <origin xyz="0 0 0" rpy="0 0 0" />
-        <geometry>
-          <mesh filename="package://reemc_description/meshes/hand/hand_finger_3_collision.stl" scale="1 1 ${-reflect * finger_reflect}" />
+          <mesh filename="package://reem_description/meshes/hand/hand_finger_3.dae" scale="1 1 ${-reflect * finger_reflect*1}" />
+        </geometry>
+        <material name="LightGrey" />
+      </visual>
+      <collision>
+        <origin xyz="0 0 0" rpy="0 0 0" />
+        <geometry>
+          <mesh filename="package://reem_description/meshes/hand/hand_finger_3_collision.stl" scale="1 1 ${-reflect * finger_reflect}" />
         </geometry>
       </collision>
@@ -158,12 +158,12 @@
         <origin xyz="0 0 0" rpy="0 0 0" />
         <geometry>
-          <mesh filename="package://reemc_description/meshes/hand/hand_palm.dae" scale="1 ${-reflect*1} 1" />
-        </geometry>
-        <material name="LightGrey" />
-      </visual>
-      <collision>
-        <origin xyz="0 0 0" rpy="0 0 0" />
-        <geometry>
-          <mesh filename="package://reemc_description/meshes/hand/hand_palm_collision.stl" scale="1 ${-reflect} 1" />
+          <mesh filename="package://reem_description/meshes/hand/hand_palm.dae" scale="1 ${-reflect*1} 1" />
+        </geometry>
+        <material name="LightGrey" />
+      </visual>
+      <collision>
+        <origin xyz="0 0 0" rpy="0 0 0" />
+        <geometry>
+          <mesh filename="package://reem_description/meshes/hand/hand_palm_collision.stl" scale="1 ${-reflect} 1" />
         </geometry>
       </collision>
@@ -189,5 +189,5 @@
       <safety_controller k_position="20"
                          k_velocity="20"
-                         soft_lower_limit="${ 0.0 * deg_to_rad + hand_eps}"
+                         soft_lower_limit="${ 0.0 * deg_to_rad}"
                          soft_upper_limit="${90.0 * deg_to_rad - hand_eps}" />
     </joint>
@@ -201,12 +201,12 @@
         <origin xyz="0 0 0" rpy="0 0 0" />
         <geometry>
-          <mesh filename="package://reemc_description/meshes/hand/hand_thumb.dae" scale="1 1 ${-reflect*1}" />
-        </geometry>
-        <material name="LightGrey" />
-      </visual>
-      <collision>
-        <origin xyz="0 0 0" rpy="0 0 0" />
-        <geometry>
-          <mesh filename="package://reemc_description/meshes/hand/hand_thumb_collision.stl" scale="1 1 ${-reflect}" />
+          <mesh filename="package://reem_description/meshes/hand/hand_thumb.dae" scale="1 1 ${-reflect}" />
+        </geometry>
+        <material name="LightGrey" />
+      </visual>
+      <collision>
+        <origin xyz="0 0 0" rpy="0 0 0" />
+        <geometry>
+          <mesh filename="package://reem_description/meshes/hand/hand_thumb_collision.stl" scale="1 1 ${-reflect}" />
         </geometry>
       </collision>

Commit message: Fix: Paths of the meshes were pointing to reem model not reemc model
git-svn-id: svn+ssh://server/srv/svn/repos/trunk/pal-ros-pkg/catkin_pkgs/reemc_robot@52210 5e370ff8-3418-0410-babe-3378cc20a00d

File: reemc_description/urdf/hand/hand.urdf.xacro (robot description, xacro)
@@ -9,7 +9,7 @@
 <robot xmlns:xacro="http://ros.org/wiki/xacro">
   <!--File includes-->
-  <xacro:include filename="$(find reem_description)/urdf/deg_to_rad.xacro" />
-  <xacro:include filename="$(find reem_description)/urdf/hand/hand.gazebo.xacro" />
-  <xacro:include filename="$(find reem_description)/urdf/hand/hand.transmission.xacro" />
+  <xacro:include filename="$(find reemc_description)/urdf/deg_to_rad.xacro" />
+  <xacro:include filename="$(find reemc_description)/urdf/hand/hand.gazebo.xacro" />
+  <xacro:include filename="$(find reemc_description)/urdf/hand/hand.transmission.xacro" />
   <!--Constant parameters-->
   <xacro:property name="hand_friction" value="0.0" /> <!--TODO: Tune-->
@@ -70,12 +70,12 @@
         <origin xyz="0 0 0" rpy="0 0 0" />
         <geometry>
-          <mesh filename="package://reem_description/meshes/hand/hand_finger_1.dae" scale="1 1 ${-reflect * finger_reflect * 1}" />
-        </geometry>
-        <material name="LightGrey" />
-      </visual>
-      <collision>
-        <origin xyz="0 0 0" rpy="0 0 0" />
-        <geometry>
-          <mesh filename="package://reem_description/meshes/hand/hand_finger_1_collision.stl" scale="1 1 ${-reflect * finger_reflect}" />
+          <mesh filename="package://reemc_description/meshes/hand/hand_finger_1.dae" scale="1 1 ${-reflect * finger_reflect * 1}" />
+        </geometry>
+        <material name="LightGrey" />
+      </visual>
+      <collision>
+        <origin xyz="0 0 0" rpy="0 0 0" />
+        <geometry>
+          <mesh filename="package://reemc_description/meshes/hand/hand_finger_1_collision.stl" scale="1 1 ${-reflect * finger_reflect}" />
         </geometry>
       </collision>
@@ -99,12 +99,12 @@
         <origin xyz="0 0 0" rpy="0 0 0" />
         <geometry>
-          <mesh filename="package://reem_description/meshes/hand/hand_finger_2.dae" scale="1 1 ${-reflect * finger_reflect * 1}" />
-        </geometry>
-        <material name="LightGrey" />
-      </visual>
-      <collision>
-        <origin xyz="0 0 0" rpy="0 0 0" />
-        <geometry>
-          <mesh filename="package://reem_description/meshes/hand/hand_finger_2_collision.stl" scale="1 1 ${-reflect * finger_reflect}" />
+          <mesh filename="package://reemc_description/meshes/hand/hand_finger_2.dae" scale="1 1 ${-reflect * finger_reflect * 1}" />
+        </geometry>
+        <material name="LightGrey" />
+      </visual>
+      <collision>
+        <origin xyz="0 0 0" rpy="0 0 0" />
+        <geometry>
+          <mesh filename="package://reemc_description/meshes/hand/hand_finger_2_collision.stl" scale="1 1 ${-reflect * finger_reflect}" />
         </geometry>
       </collision>
@@ -128,12 +128,12 @@
         <origin xyz="0 0 0" rpy="0 0 0" />
         <geometry>
-          <mesh filename="package://reem_description/meshes/hand/hand_finger_3.dae" scale="1 1 ${-reflect * finger_reflect*1}" />
-        </geometry>
-        <material name="LightGrey" />
-      </visual>
-      <collision>
-        <origin xyz="0 0 0" rpy="0 0 0" />
-        <geometry>
-          <mesh filename="package://reem_description/meshes/hand/hand_finger_3_collision.stl" scale="1 1 ${-reflect * finger_reflect}" />
+          <mesh filename="package://reemc_description/meshes/hand/hand_finger_3.dae" scale="1 1 ${-reflect * finger_reflect*1}" />
+        </geometry>
+        <material name="LightGrey" />
+      </visual>
+      <collision>
+        <origin xyz="0 0 0" rpy="0 0 0" />
+        <geometry>
+          <mesh filename="package://reemc_description/meshes/hand/hand_finger_3_collision.stl" scale="1 1 ${-reflect * finger_reflect}" />
         </geometry>
       </collision>
@@ -158,12 +158,12 @@
         <origin xyz="0 0 0" rpy="0 0 0" />
         <geometry>
-          <mesh filename="package://reem_description/meshes/hand/hand_palm.dae" scale="1 ${-reflect*1} 1" />
-        </geometry>
-        <material name="LightGrey" />
-      </visual>
-      <collision>
-        <origin xyz="0 0 0" rpy="0 0 0" />
-        <geometry>
-          <mesh filename="package://reem_description/meshes/hand/hand_palm_collision.stl" scale="1 ${-reflect} 1" />
+          <mesh filename="package://reemc_description/meshes/hand/hand_palm.dae" scale="1 ${-reflect*1} 1" />
+        </geometry>
+        <material name="LightGrey" />
+      </visual>
+      <collision>
+        <origin xyz="0 0 0" rpy="0 0 0" />
+        <geometry>
+          <mesh filename="package://reemc_description/meshes/hand/hand_palm_collision.stl" scale="1 ${-reflect} 1" />
         </geometry>
       </collision>
@@ -201,12 +201,12 @@
         <origin xyz="0 0 0" rpy="0 0 0" />
         <geometry>
-          <mesh filename="package://reem_description/meshes/hand/hand_thumb.dae" scale="1 1 ${-reflect}" />
-        </geometry>
-        <material name="LightGrey" />
-      </visual>
-      <collision>
-        <origin xyz="0 0 0" rpy="0 0 0" />
-        <geometry>
-          <mesh filename="package://reem_description/meshes/hand/hand_thumb_collision.stl" scale="1 1 ${-reflect}" />
+          <mesh filename="package://reemc_description/meshes/hand/hand_thumb.dae" scale="1 1 ${-reflect}" />
+        </geometry>
+        <material name="LightGrey" />
+      </visual>
+      <collision>
+        <origin xyz="0 0 0" rpy="0 0 0" />
+        <geometry>
+          <mesh filename="package://reemc_description/meshes/hand/hand_thumb_collision.stl" scale="1 1 ${-reflect}" />
         </geometry>
       </collision>
