Commit message: Replaced hands with boxes

File: reemc_description/urdf/hand/hand.urdf.xacro (robot description, xacro)
@@ -17,129 +17,4 @@
   <xacro:property name="hand_max_vel"  value="2.0" />
   <xacro:property name="hand_eps"      value="0.02" />
-  <xacro:macro name="reem_finger" params="hand_name hand_side hand_reflect finger_name finger_reflect">
-    <!-- Actuated joint -->
-    <joint name="${hand_name}_${hand_side}_${finger_name}_joint" type="revolute">
-      <parent link="${hand_name}_${hand_side}_palm_link" />
-      <child link="${hand_name}_${hand_side}_${finger_name}_link" />
-      <origin xyz="0.101 ${reflect * 0.0025} ${finger_reflect * 0.0165}" rpy="${(90.0 - reflect * 90.0) * deg_to_rad} 0 ${reflect * 90.0 * deg_to_rad}" />
-      <axis xyz="0 0 1" />
-      <limit lower="${0.0 * deg_to_rad}" upper="${250.0 * deg_to_rad}" effort="2.0" velocity="${hand_max_vel}" /> <!-- TODO: Tune values -->
-      <dynamics friction="${hand_friction}" damping="${hand_damping}"/>
-      <safety_controller k_position="20"
-                         k_velocity="20"
-                         soft_lower_limit="${  0.0 * deg_to_rad}"
-                         soft_upper_limit="${250.0 * deg_to_rad - hand_eps}" />
-    </joint>
-    <link name="${hand_name}_${hand_side}_${finger_name}_link">
-      <inertial>
-        <origin xyz="0.00175 -0.01837 -0.00198" rpy="0 0 0" />
-        <mass value="0.055" />
-        <inertia ixx="0.00001450121"  ixy="-0.00000065488"  ixz="-0.00000039654" iyy="0.0000072995" iyz="0.00000012168" izz="0.00001262409" />
-      </inertial>
-      <visual>
-        <origin xyz="0 0 0" rpy="0 0 0" />
-        <geometry>
-          <sphere radius="0.001"/>
-        </geometry>
-        <material name="LightGrey" />
-      </visual>
-      <collision>
-        <origin xyz="0 0 0" rpy="0 0 0" />
-        <geometry>
-          <sphere radius="0.001"/>
-        </geometry>
-      </collision>
-    </link>
-    <!-- Read-only phalanxes-->
-    <joint name="${hand_name}_${hand_side}_${finger_name}_1_joint" type="revolute">
-      <parent link="${hand_name}_${hand_side}_palm_link" />
-      <child link="${hand_name}_${hand_side}_${finger_name}_1_link" />
-      <origin xyz="0.101 ${reflect * 0.0025} ${finger_reflect * 0.0165}" rpy="${(90.0 - reflect * 90.0) * deg_to_rad} 0 ${reflect * 90.0 * deg_to_rad}" />
-      <axis xyz="0 0 1" />
-      <limit lower="${0.0 * deg_to_rad}" upper="${90.0 * deg_to_rad}" effort="2.0" velocity="${hand_max_vel}" />
-      <dynamics friction="${hand_friction}" damping="${hand_damping}"/>
-      <mimic joint="${hand_name}_${hand_side}_${finger_name}_joint" multiplier="${90.0 / 250.0}" offset="0.0" />
-    </joint>
-    <link name="${hand_name}_${hand_side}_${finger_name}_1_link">
-      <inertial>
-        <origin xyz="0.00175 -0.01837 -0.00198" rpy="0 0 0" />
-        <mass value="0.055" />
-        <inertia ixx="0.00001450121"  ixy="-0.00000065488"  ixz="-0.00000039654" iyy="0.0000072995" iyz="0.00000012168" izz="0.00001262409" />
-      </inertial>
-      <visual>
-        <origin xyz="0 0 0" rpy="0 0 0" />
-        <geometry>
-          <mesh filename="package://reemc_description/meshes/hand/hand_finger_1.dae" scale="1 1 ${-reflect * finger_reflect * 1}" />
-        </geometry>
-        <material name="LightGrey" />
-      </visual>
-      <collision>
-        <origin xyz="0 0 0" rpy="0 0 0" />
-        <geometry>
-          <mesh filename="package://reemc_description/meshes/hand/hand_finger_1_collision.stl" scale="1 1 ${-reflect * finger_reflect}" />
-        </geometry>
-      </collision>
-    </link>
-    <joint name="${hand_name}_${hand_side}_${finger_name}_2_joint" type="revolute">
-      <parent link="${hand_name}_${hand_side}_${finger_name}_1_link" />
-      <child link="${hand_name}_${hand_side}_${finger_name}_2_link" />
-      <origin xyz="0.00357 -0.04084 0" rpy="0 0 0" />
-      <axis xyz="0 0 1" />
-      <limit lower="${0.0 * deg_to_rad}" upper="${80.0 * deg_to_rad}" effort="1.0" velocity="${hand_max_vel}" />
-      <dynamics friction="${hand_friction}" damping="${hand_damping}"/>
-      <mimic joint="${hand_name}_${hand_side}_${finger_name}_joint" multiplier="${80.0 / 250.0}" offset="0.0" />
-    </joint>
-    <link name="${hand_name}_${hand_side}_${finger_name}_2_link">
-      <inertial>
-        <origin xyz="0.00181 -0.01275 -0.00064" rpy="0 0 0" />
-        <mass value="0.02972" />
-        <inertia ixx="0.00000428193"  ixy="-0.00000049978"  ixz="-0.00000002985" iyy="0.00000254434" iyz="0.00000007762" izz="0.00000345152" />
-      </inertial>
-      <visual>
-        <origin xyz="0 0 0" rpy="0 0 0" />
-        <geometry>
-          <mesh filename="package://reemc_description/meshes/hand/hand_finger_2.dae" scale="1 1 ${-reflect * finger_reflect * 1}" />
-        </geometry>
-        <material name="LightGrey" />
-      </visual>
-      <collision>
-        <origin xyz="0 0 0" rpy="0 0 0" />
-        <geometry>
-          <mesh filename="package://reemc_description/meshes/hand/hand_finger_2_collision.stl" scale="1 1 ${-reflect * finger_reflect}" />
-        </geometry>
-      </collision>
-    </link>
-    <joint name="${hand_name}_${hand_side}_${finger_name}_3_joint" type="revolute">
-      <parent link="${hand_name}_${hand_side}_${finger_name}_2_link" />
-      <child link="${hand_name}_${hand_side}_${finger_name}_3_link" />
-      <origin xyz="0.00572 -0.0269 0" rpy="0 0 0" />
-      <axis xyz="0 0 1" />
-      <limit lower="${0.0 * deg_to_rad}" upper="${80.0 * deg_to_rad}" effort="1.0" velocity="${hand_max_vel}" />
-      <dynamics friction="${hand_friction}" damping="${hand_damping}"/>
-      <mimic joint="${hand_name}_${hand_side}_${finger_name}_joint" multiplier="${80.0 / 250.0}" offset="0.0" />
-    </joint>
-    <link name="${hand_name}_${hand_side}_${finger_name}_3_link">
-      <inertial>
-        <origin xyz="0 -0.00704 0.00019" rpy="0 0 0" />
-        <mass value="0.01522" />
-        <inertia ixx="0.00000128478"  ixy="-0.00000008056"  ixz="-0.00000001698" iyy="0.00000080139" iyz="-0.00000002884" izz="0.00000090928" />
-      </inertial>
-      <visual>
-        <origin xyz="0 0 0" rpy="0 0 0" />
-        <geometry>
-          <mesh filename="package://reemc_description/meshes/hand/hand_finger_3.dae" scale="1 1 ${-reflect * finger_reflect*1}" />
-        </geometry>
-        <material name="LightGrey" />
-      </visual>
-      <collision>
-        <origin xyz="0 0 0" rpy="0 0 0" />
-        <geometry>
-          <mesh filename="package://reemc_description/meshes/hand/hand_finger_3_collision.stl" scale="1 1 ${-reflect * finger_reflect}" />
-        </geometry>
-      </collision>
-    </link>
-    <xacro:hand_finger_gazebo finger_name="${hand_name}_${hand_side}_${finger_name}"/>
-    <xacro:hand_finger_transmission finger_name="${hand_name}_${hand_side}_${finger_name}" actuator_reduction="1"/>
-  </xacro:macro>
   <xacro:macro name="reem_hand" params="name parent side reflect">
     <!-- Palm -->
@@ -147,25 +22,57 @@
       <parent link="${parent}" />
       <child link="${name}_${side}_palm_link" />
-      <origin xyz="0 0 0" rpy="0 0 0" />
+      <origin xyz="0 0 0" rpy="${reflect*1.57} 0 0" />
     </joint>
     <link name="${name}_${side}_palm_link">
       <inertial>
-        <origin xyz="0.05904 ${-reflect * 0.00925} -0.00075 " rpy="0 0 0" /> <!--TODO: This does not make sense!, there must be a bug in how Gazebo bungles the CoM of a chain of fixed joints-->
+        <origin xyz="0.1 0 0" rpy="0 0 0" />
         <mass value="0.68275" />
         <inertia ixx="0.00045643484"  ixy="0.00001885321"  ixz="-0.0000103596" iyy="0.00076077407" iyz="-0.00000266311" izz="0.00052521525" />
       </inertial>
       <visual>
-        <origin xyz="0 0 0" rpy="0 0 0" />
+        <origin xyz="0.1 0 0" rpy = "0 0 0"/>
         <geometry>
-          <mesh filename="package://reemc_description/meshes/hand/hand_palm.dae" scale="1 ${-reflect*1} 1" />
+          <box size="0.2 0.1 0.025" />
         </geometry>
-        <material name="LightGrey" />
       </visual>
       <collision>
-        <origin xyz="0 0 0" rpy="0 0 0" />
+        <origin xyz="0.1 0 0" rpy = "0 0 0"/>
         <geometry>
-          <mesh filename="package://reemc_description/meshes/hand/hand_palm_collision.stl" scale="1 ${-reflect} 1" />
+          <box size="0.2 0.1 0.025" />
         </geometry>
       </collision>
+    </link>
+    <joint name="${name}_${side}_end_effector_joint" type="fixed">
+      <parent link="${name}_${side}_palm_link"/>
+      <child link="${name}_${side}_end_effector_link"/>
+      <origin xyz="0.1 0 -0.0125" rpy="0 0 0" />
+    </joint>
+    <link name="${name}_${side}_end_effector_link">
+      <inertial>
+        <origin xyz="0 0 0" rpy="0 0 0" />
+        <mass value="0" />
+        <inertia ixx="0"  ixy="0"  ixz="0" iyy="0" iyz="0" izz="0" />
+      </inertial>
+    </link>
+    <joint name="${name}_${side}_indication_joint" type="fixed">
+      <parent link="${name}_${side}_palm_link"/>
+      <child link="${name}_${side}_indication_link"/>
+      <origin xyz="0.1 0 0.0125" rpy="0 0 0" />
+    </joint>
+    <link name="${name}_${side}_indication_link">
+      <inertial>
+        <origin xyz="0 0 -0.0125" rpy="${reflect*1.57} 0 0" />
+        <mass value="0.0" />
+        <inertia ixx="0"  ixy="0"  ixz="0" iyy="0" iyz="0" izz="0" />
+      </inertial>
+      <visual>
+        <origin xyz="0 0 0.0125" rpy="0 0 0" />
+        <geometry>
+          <cylinder length="0.02" radius="0.01"/>
+        </geometry>
+        <material name = "">
+          <color rgba="0 0.5 0 1.0"></color>
+        </material>
+      </visual>
     </link>
     <gazebo reference="${name}_${side}_palm_link">
@@ -178,73 +85,4 @@
      <minDepth>0.00</minDepth>
     </gazebo>
-    <xacro:hand_gazebo name="${name}_${side}_palm"/>
-    <!-- Thumb -->
-    <joint name="${name}_${side}_thumb_joint" type="revolute">
-      <parent link="${name}_${side}_palm_link" />
-      <child link="${name}_${side}_thumb_link" />
-      <origin xyz="0.03649 ${reflect * 0.008}  0.02" rpy="${(90.0 + reflect * 90.0) * deg_to_rad} ${(90.0 + 13) * deg_to_rad} ${reflect * 13.0 * deg_to_rad}" />
-      <axis xyz="0 0 1" />
-      <limit lower="${0.0 * deg_to_rad}" upper="${90.0 * deg_to_rad}" effort="2.0" velocity="${hand_max_vel}" />
-      <dynamics friction="${hand_friction}" damping="${hand_damping}"/>
-      <safety_controller k_position="20"
-                         k_velocity="20"
-                         soft_lower_limit="${ 0.0 * deg_to_rad}"
-                         soft_upper_limit="${90.0 * deg_to_rad - hand_eps}" />
-    </joint>
-    <link name="${name}_${side}_thumb_link">
-      <inertial>
-        <origin xyz="0.00049 0.00451 ${-reflect*0.04179}" rpy="0 0 0" />
-        <mass value="0.07088" />
-        <inertia ixx="0.0000699364"  ixy="0.00000345915"  ixz="0.00000425008" iyy="0.00002675459" iyz="0.00002381865" izz="0.00004787167" />
-      </inertial>
-      <visual>
-        <origin xyz="0 0 0" rpy="0 0 0" />
-        <geometry>
-          <mesh filename="package://reemc_description/meshes/hand/hand_thumb.dae" scale="1 1 ${-reflect}" />
-        </geometry>
-        <material name="LightGrey" />
-      </visual>
-      <collision>
-        <origin xyz="0 0 0" rpy="0 0 0" />
-        <geometry>
-          <mesh filename="package://reemc_description/meshes/hand/hand_thumb_collision.stl" scale="1 1 ${-reflect}" />
-        </geometry>
-      </collision>
-    </link>
-    <gazebo reference="${name}_${side}_thumb_link">
-     <kp>1000000.0</kp>
-     <kd>100.0</kd>
-     <mu1>1.0</mu1>
-     <mu2>1.0</mu2>
-     <fdir1>0 0 1</fdir1>
-     <maxVel>1.0</maxVel>
-     <minDepth>0.00</minDepth>
-    </gazebo>
-    <gazebo reference="${name}_${side}_thumb_joint">
-       <implicitSpringDamper>1</implicitSpringDamper>
-    </gazebo>
-    <!-- Grasping frame -->
-    <!-- grasp planner will approach along x-axis -->
-    <joint name="${name}_${side}_grasping_frame_joint" type="fixed">
-      <parent link="${name}_${side}_palm_link" />
-      <child link="${name}_${side}_grasping_frame" />
-      <origin xyz="0.055 ${reflect * 0.054} 0.018" rpy="0 0 0" />
-    </joint>
-    <link name="${name}_${side}_grasping_frame">
-      <inertial>
-        <origin xyz="0 0 0" rpy="0 0 0" />
-        <mass value="0.01" /> <!-- matrix below must not be zero, or Gazebo won't load -->
-        <inertia ixx="0.00001" ixy="0.0" ixz="0.0"
-                 iyy="0.00001" iyz="0.0"
-                 izz="0.00001" />
-      </inertial>
-    </link>
-    <xacro:hand_thumb_transmission name="${name}_${side}_thumb" reduction="1" />
-    <!-- Index finger -->
-    <xacro:reem_finger hand_name="${name}" hand_side="${side}" hand_reflect="${reflect}" finger_name="index" finger_reflect="1"/>
-    <!-- Middle finger -->
-    <xacro:reem_finger hand_name="${name}" hand_side="${side}" hand_reflect="${reflect}" finger_name="middle" finger_reflect="-1"/>
-    <!-- grasping hack -->
-    <xacro:hand_grasping_hack side="${side}" />
   </xacro:macro>
 </robot>

File: reemc_description/urdf/leg/leg.urdf.xacro (robot description, xacro)
@@ -190,5 +190,5 @@
         <origin rpy="0 0 0" xyz="0.1 ${-reflect*0.01} 0.025 "/>
         <geometry>
-          <box size="0.02 0.14 0.210"/>
+          <box size="0.03 0.14 0.210"/>
         </geometry>
       </collision>

File: reemc_description/urdf/torso/torso.urdf.xacro (robot description, xacro)
@@ -34,5 +34,5 @@
       </visual>
     </link>
-    <joint name="${name}_1_joint" type="revolute">
+    <joint name="${name}_1_joint" type="fixed">
       <parent link="${parent}"/>
       <child link="${name}_1_link"/>
@@ -70,5 +70,5 @@
       </collision>
     </link>
-    <joint name="${name}_2_joint" type="revolute">
+    <joint name="${name}_2_joint" type="fixed">
       <parent link="${name}_1_link" />
       <child link="${name}_2_link" />
