Commit message: reemc_description: remove initial pose (overwritten anyway)

File: reemc_description/robots/reemc_full.urdf.xacro (robot description, xacro)
@@ -30,9 +30,5 @@
       </geometry>
     </collision>
- </link>
- <gazebo>
-    <!-- robot model offset -->
-    <pose>0 0 0.85 0 0 0</pose>
-  </gazebo>
+  </link>
   <!-- The following included files set up definitions of parts of the robot body -->
   <xacro:include filename="$(find reemc_description)/urdf/leg/leg.urdf.xacro" />

Commit message: Merge reemc_description from OROCOS_2.X
git-svn-id: svn+ssh://server/srv/svn/repos/branches/hydro_migration/pal-ros-pkg/catkin_pkgs/reemc_robot@49866 5e370ff8-3418-0410-babe-3378cc20a00d

File: reemc_description/robots/reemc_full.urdf.xacro (robot description, xacro)
@@ -71,4 +71,6 @@
   </xacro:reemc_back_camera>
   <!-- imu -->
-  <xacro:reemc_imu name="imu" parent="base_link" update_rate="100.0"/>
+  <xacro:reemc_imu name="imu" parent="base_link" update_rate="100.0">
+    <origin xyz="0 0 0" rpy="${180.0*deg_to_rad} 0 0"/>
+  </xacro:reemc_imu>
 </robot>

File: reemc_description/robots/reemc_lower_body.urdf.xacro (robot description, xacro)
@@ -59,4 +59,6 @@
   <xacro:reemc_leg  name="leg" side="left" reflect="-1.0" parent="base_link"/>
   <!-- imu -->
-  <xacro:reemc_imu name="imu" parent="base_link" update_rate="1000.0"/>
+  <xacro:reemc_imu name="imu" parent="base_link" update_rate="100.0">
+    <origin xyz="0 0 0" rpy="${180*deg_to_rad} 0 0"/>
+  </xacro:reemc_imu>
 </robot>

File: reemc_description/urdf/leg/leg.urdf.xacro (robot description, xacro)
@@ -215,5 +215,5 @@
     <joint name="${side}_sole_joint" type="fixed">
       <!-- origin x taken from link_${side}_6_link/visual/origin/x above -->
-      <origin xyz="0.110 0.0 0.0" rpy="0.0 ${-90.0 * deg_to_rad} 0.0"/>
+      <origin xyz="0.117 0.0 0.0" rpy="0.0 ${-90.0 * deg_to_rad} 0.0"/>
       <axis xyz="0 0 1"/>
       <parent link="leg_${side}_6_link"/>
@@ -281,5 +281,5 @@
     <xacro:reemc_leg_simple_transmission name="${name}" side="${side}" number="6" reduction="${leg_reduction}" />
    <xacro:reemc_laser name="${side}_laser" parent="${side}_sole_link" ros_topic="${side}_scan" update_rate="10.0" min_angle="${-90*deg_to_rad}" max_angle="${90*deg_to_rad}" nrays="360" >
-     <origin xyz="${0.170 -0.085} ${0.071 -((1+reflect)*0.01 + 0.061)} ${0.04}" rpy="0.0 0.0 ${-30.0*reflect*deg_to_rad}" />
+     <origin xyz="${0.170 -0.085} ${0.071 -((1+reflect)*0.01 + 0.061)} ${0.073}" rpy="0.0 0.0 ${-30.0*reflect*deg_to_rad}" />
     </xacro:reemc_laser>
   </xacro:macro>

File: reemc_description/urdf/sensors/imu.urdf.xacro (robot description, xacro)
@@ -8,5 +8,5 @@
 -->
 <robot name="reemc" xmlns:xacro="http://ros.org/wiki/xacro">
-  <xacro:macro name="reemc_imu" params="name parent update_rate">
+  <xacro:macro name="reemc_imu" params="name parent update_rate *origin">
     <link name="${name}_link">
       <inertial>
@@ -23,7 +23,7 @@
     </link>
     <joint name="imu_joint" type="fixed">
+      <insert_block name="origin"/>
       <parent link="${parent}"/>
       <child link="${name}_link"/>
-      <origin xyz="0.0 0 0.0" rpy="0 0 0"/>
     </joint>
   </xacro:macro>

Commit message: Updated the reemc_description to our local changes, mainly urdf little changes

File: reemc_description/robots/reemc_full.urdf.xacro (robot description, xacro)
@@ -1,5 +1,5 @@
 <?xml version="1.0"?>
 <!--
-  Copyright (c) 2011, PAL Robotics, S.L.
+  Copyright (c) 2013, PAL Robotics, S.L.
   All rights reserved.
   This work is licensed under the Creative Commons Attribution-NonCommercial-NoDerivs 3.0 Unported License.
@@ -62,13 +62,15 @@
   <!-- stereo camera -->
   <!-- IMPORTANT: focal_length = image_width/(2tan(hfov/2)) -->
-  <xacro:reemc_stereo_camera parent="head_2_link" name="stereo" focal_length="461.941850" hfov="${71.0*deg_to_rad}" image_format="B8G8R8" image_width="659" image_height="493">
+  <xacro:reemc_stereo_camera parent="head_2_link" name="stereo" focal_length="461.943804" hfov="${71.0*deg_to_rad}" image_format="B8G8R8" image_width="659" image_height="493">
 <!-- The following transformations expresses the pose of the stereo_link (X pointing forward, Z upwards and Y leftwards, contrary to the stereo_optical_link which has Z pointing forward) wrt  head_2_link. -->
     <origin xyz="0.08203  -0.0935  0.0365" rpy="1.56293 -0.00855922 -0.0201307" />
   </xacro:reemc_stereo_camera>
-  <xacro:reemc_back_camera parent="torso_2_link" name="back_camera" focal_length="376.003507" hfov="${89.999451423*deg_to_rad}" image_format="B8G8R8" image_width="752" image_height="480" >
+  <xacro:reemc_back_camera parent="torso_2_link" name="back_camera" focal_length="376.002379" hfov="${89.999451423*deg_to_rad}" image_format="B8G8R8" image_width="752" image_height="480" >
     <!-- The following transformations expresses the pose of the back_camera_link (X pointing forward, Z upwards and Y leftwards, contrary to the stereo_optical_link which has Z pointing forward) wrt  torso_2_link. -->
     <origin xyz="-0.128 -0.317 0" rpy="${-90.0*deg_to_rad} 0 ${180.0*deg_to_rad}" />
   </xacro:reemc_back_camera>
   <!-- imu -->
-  <xacro:reemc_imu name="imu" parent="base_link" update_rate="100.0"/>
+  <xacro:reemc_imu name="imu" parent="base_link" update_rate="100.0">
+    <origin xyz="0 0 0" rpy="${180.0*deg_to_rad} 0 0"/>
+  </xacro:reemc_imu>
 </robot>

File: reemc_description/urdf/sensors/ftsensor.gazebo.xacro (robot description, xacro)
@@ -12,14 +12,14 @@
     <sensor name="${name}_contact_sensor" type="contact">
       <pose>0.105 0.071 0 0 0 0</pose>
-       <always_on>1</always_on>
-       <update_rate>${update_rate}</update_rate>
-       <contact>
-         <collision>${name}_collision</collision>
-       </contact>
-   </sensor>
-</gazebo>
-<gazebo reference="${name}">
-  <provideFeedback>1</provideFeedback>
-</gazebo>
+      <always_on>1</always_on>
+      <update_rate>${update_rate}</update_rate>
+      <contact>
+        <collision>${name}_collision</collision>
+      </contact>
+    </sensor>
+  </gazebo>
+  <gazebo reference="${name}">
+    <provideFeedback>1</provideFeedback>
+  </gazebo>
 </xacro:macro>
 </robot>

File: reemc_description/urdf/sensors/range.gazebo.xacro (robot description, xacro)
@@ -35,5 +35,5 @@
           </range>
         </ray>
-        <plugin filename="libgazebo_ros_laser.so" name="gazebo_ros_laser">
+        <plugin filename="libgazebo_ros_range.so" name="gazebo_ros_range">
           <gaussianNoise>0.005</gaussianNoise>
           <alwaysOn>true</alwaysOn>

Commit message: Updated model in sync with PAL local package.
- Separated a part of the launch in reemc_bringup.launch
- Added config dir on install
- cmfDamping -> implicitSpringDamper
- Removed collision groups (not supported).
- Updated copyrights.
- Updated some params slightly.

File: reemc_description/robots/reemc_full.urdf.xacro (robot description, xacro)
@@ -1,5 +1,5 @@
 <?xml version="1.0"?>
 <!--
-  Copyright (c) 2011, PAL Robotics, S.L.
+  Copyright (c) 2014, PAL Robotics, S.L.
   All rights reserved.
   This work is licensed under the Creative Commons Attribution-NonCommercial-NoDerivs 3.0 Unported License.
@@ -62,13 +62,15 @@
   <!-- stereo camera -->
   <!-- IMPORTANT: focal_length = image_width/(2tan(hfov/2)) -->
-  <xacro:reemc_stereo_camera parent="head_2_link" name="stereo" focal_length="461.941850" hfov="${71.0*deg_to_rad}" image_format="B8G8R8" image_width="659" image_height="493">
+  <xacro:reemc_stereo_camera parent="head_2_link" name="stereo" focal_length="461.943804" hfov="${71.0*deg_to_rad}" image_format="B8G8R8" image_width="659" image_height="493">
 <!-- The following transformations expresses the pose of the stereo_link (X pointing forward, Z upwards and Y leftwards, contrary to the stereo_optical_link which has Z pointing forward) wrt  head_2_link. -->
     <origin xyz="0.08203  -0.0935  0.0365" rpy="1.56293 -0.00855922 -0.0201307" />
   </xacro:reemc_stereo_camera>
-  <xacro:reemc_back_camera parent="torso_2_link" name="back_camera" focal_length="376.003507" hfov="${89.999451423*deg_to_rad}" image_format="B8G8R8" image_width="752" image_height="480" >
+  <xacro:reemc_back_camera parent="torso_2_link" name="back_camera" focal_length="376.002379" hfov="${89.999451423*deg_to_rad}" image_format="B8G8R8" image_width="752" image_height="480" >
     <!-- The following transformations expresses the pose of the back_camera_link (X pointing forward, Z upwards and Y leftwards, contrary to the stereo_optical_link which has Z pointing forward) wrt  torso_2_link. -->
     <origin xyz="-0.128 -0.317 0" rpy="${-90.0*deg_to_rad} 0 ${180.0*deg_to_rad}" />
   </xacro:reemc_back_camera>
   <!-- imu -->
-  <xacro:reemc_imu name="imu" parent="base_link" update_rate="100.0"/>
+  <xacro:reemc_imu name="imu" parent="base_link" update_rate="100.0">
+    <origin xyz="0 0 0" rpy="${180.0*deg_to_rad} 0 0"/>
+  </xacro:reemc_imu>
 </robot>

File: reemc_description/robots/reemc_lower_body.urdf.xacro (robot description, xacro)
@@ -1,5 +1,5 @@
 <?xml version="1.0"?>
 <!--
-  Copyright (c) 2011, PAL Robotics, S.L.
+  Copyright (c) 2014, PAL Robotics, S.L.
   All rights reserved.
   This work is licensed under the Creative Commons Attribution-NonCommercial-NoDerivs 3.0 Unported License.
@@ -59,4 +59,6 @@
   <xacro:reemc_leg  name="leg" side="left" reflect="-1.0" parent="base_link"/>
   <!-- imu -->
-  <xacro:reemc_imu name="imu" parent="base_link" update_rate="1000.0"/>
+  <xacro:reemc_imu name="imu" parent="base_link" update_rate="100.0">
+    <origin xyz="0 0 0" rpy="${180*deg_to_rad} 0 0"/>
+  </xacro:reemc_imu>
 </robot>

File: reemc_description/urdf/sensors/stereo_camera.urdf.xacro (robot description, xacro)
@@ -1,5 +1,5 @@
 <?xml version="1.0"?>
 <!--
-  Copyright (c) 2011, PAL Robotics, S.L.
+  Copyright (c) 2014, PAL Robotics, S.L.
   All rights reserved.
   This work is licensed under the Creative Commons Attribution-NonCommercial-NoDerivs 3.0 Unported License.

Commit message: Add ft sensor to the wrist and Hey5 hand

File: reemc_description/robots/reemc_full.urdf.xacro (robot description, xacro)
@@ -40,5 +40,6 @@
   <xacro:include filename="$(find reemc_description)/urdf/arm/arm.urdf.xacro" />
   <!-- Hand -->
-  <xacro:include filename="$(find reemc_description)/urdf/hand/hand.urdf.xacro" />
+<!--  <xacro:include filename="$(find reemc_description)/urdf/hand/hand.urdf.xacro" /> -->
+  <xacro:include filename="$(find hey5_description)/urdf/hey5_hand.urdf.xacro" />
   <!-- Sensors -->
   <xacro:include filename="$(find reemc_description)/urdf/sensors/imu.urdf.xacro" />
@@ -46,4 +47,5 @@
   <xacro:include filename="$(find reemc_description)/urdf/sensors/stereo_camera.urdf.xacro" />
   <xacro:include filename="$(find reemc_description)/urdf/sensors/back_camera.urdf.xacro" />
+  <xacro:include filename="$(find reemc_description)/urdf/sensors/ftsensor.urdf.xacro" />
   <!-- Generic simulator_gazebo plugins -->
   <xacro:include filename="$(find reemc_description)/gazebo/gazebo.urdf.xacro" />
@@ -58,6 +60,20 @@
   <xacro:reem_arm name="arm" parent="torso_2_link" side="right" reflect="1.0"  />
   <xacro:reem_arm name="arm" parent="torso_2_link" side="left"  reflect="-1.0" />
-  <xacro:reem_hand name="hand" parent="arm_right_tool_link" side="right" reflect="1.0"  />
-  <xacro:reem_hand name="hand" parent="arm_left_tool_link"  side="left"  reflect="-1.0" />
+<!--
+  <xacro:ft_sensor name="wrist" parent="arm_right_tool_link" side="right" reflect="1.0"  />
+  <xacro:ft_sensor name="wrist" parent="arm_left_tool_link"  side="left"  reflect="-1.0" />
+-->
+<!--
+  <xacro:reem_hand name="hand" parent="wrist_right_ft_tool_link" side="right" reflect="1.0"  />
+  <xacro:reem_hand name="hand" parent="wrist_left_ft_tool_link"  side="left"  reflect="-1.0" />
+-->
+<!--
+  <xacro:hey5_hand parent="wrist_right_ft_tool_link" name="hand_right" reflect="1" >
+    <origin xyz="0 0 0" rpy="0 0 0" />
+  </xacro:hey5_hand>
+  <xacro:hey5_hand parent="wrist_left_ft_tool_link" name="hand_left" reflect="-1" >
+    <origin xyz="0 0 0" rpy="${180 * deg_to_rad} 0 0" />
+  </xacro:hey5_hand>
+-->
   <!-- stereo camera -->
   <!-- IMPORTANT: focal_length = image_width/(2tan(hfov/2)) -->

File: reemc_description/urdf/arm/wrist.urdf.xacro (robot description, xacro)
@@ -152,4 +152,5 @@
     <gazebo reference="${name}_${side}_7_joint">
         <implicitSpringDamper>1</implicitSpringDamper>
+        <provideFeedback>1</provideFeedback>
     </gazebo>
     <!-- extensions -->

File: reemc_description/urdf/hand/hand.urdf.xacro (robot description, xacro)
@@ -147,4 +147,5 @@
       <parent link="${parent}" />
       <child link="${name}_${side}_palm_link" />
+<!--      <origin xyz="0 0 0" rpy="${-90.0 * deg_to_rad} ${-90.0 * deg_to_rad} 0" /> -->
       <origin xyz="0 0 0" rpy="0 0 0" />
     </joint>

Commit message: Parametrized wrist joint 6 limit to support different joint limits on reemc with ft sensor

File: reemc_description/robots/reemc_full.urdf.xacro (robot description, xacro)
@@ -56,6 +56,6 @@
   <xacro:reem_torso name="torso" parent="base_link"/>
   <xacro:reem_head  name="head"  parent="torso_2_link"/>
-  <xacro:reem_arm name="arm" parent="torso_2_link" side="right" reflect="1.0"  />
-  <xacro:reem_arm name="arm" parent="torso_2_link" side="left"  reflect="-1.0" />
+  <xacro:reem_arm name="arm" parent="torso_2_link" side="right" reflect="1.0" wrist_6_range="90.0" />
+  <xacro:reem_arm name="arm" parent="torso_2_link" side="left"  reflect="-1.0" wrist_6_range="90.0" />
   <xacro:reem_hand name="hand" parent="arm_right_tool_link" side="right" reflect="1.0"  />
   <xacro:reem_hand name="hand" parent="arm_left_tool_link"  side="left"  reflect="-1.0" />

File: reemc_description/robots/reemc_full_ft_hey5.urdf.xacro (robot description, xacro)
@@ -57,6 +57,6 @@
   <xacro:reem_torso name="torso" parent="base_link"/>
   <xacro:reem_head  name="head"  parent="torso_2_link"/>
-  <xacro:reem_arm name="arm" parent="torso_2_link" side="right" reflect="1.0"  />
-  <xacro:reem_arm name="arm" parent="torso_2_link" side="left"  reflect="-1.0" />
+  <xacro:reem_arm name="arm" parent="torso_2_link" side="right" reflect="1.0" wrist_6_range="81"/>
+  <xacro:reem_arm name="arm" parent="torso_2_link" side="left"  reflect="-1.0" wrist_6_range="81"/>
   <xacro:ft_sensor name="wrist" parent="arm_right_tool_link" side="right" reflect="1.0"  />
   <xacro:ft_sensor name="wrist" parent="arm_left_tool_link"  side="left"  reflect="-1.0" />

File: reemc_description/urdf/arm/arm.urdf.xacro (robot description, xacro)
@@ -25,5 +25,5 @@
   <xacro:property name="arm_eps"            value="0.02" />
   <!-- TODO: Update dynamic models -->
-  <xacro:macro name="reem_arm" params="name parent side reflect">
+  <xacro:macro name="reem_arm" params="name parent side reflect wrist_6_range">
     <!--************************-->
     <!--        SHOULDER        -->
@@ -202,5 +202,5 @@
     <!--        WRIST           -->
     <!--************************-->
-    <xacro:reem_wrist name="arm" parent="${name}_${side}_4_link" side="${side}" reflect="${reflect}"  />
+    <xacro:reem_wrist name="arm" parent="${name}_${side}_4_link" side="${side}" reflect="${reflect}" wrist_6_range="${wrist_6_range}" />
     <!--***********************-->
     <!--        TOOL           -->

File: reemc_description/urdf/arm/wrist.urdf.xacro (robot description, xacro)
@@ -22,5 +22,5 @@
   <xacro:property name="wrist_eps"          value="0.02" />
   <!-- TODO: Update dynamic models -->
-  <xacro:macro name="reem_wrist" params="name parent side reflect">
+  <xacro:macro name="reem_wrist" params="name parent side reflect wrist_6_range">
     <!--************************-->
     <!--        WRIST           -->
@@ -89,10 +89,10 @@
       <origin xyz="0 0 ${0.15 * reflect}" rpy="${-90.0 * reflect * deg_to_rad} 0 0" />
       <axis xyz="0 0 1" />
-      <limit lower="${-90.0 * deg_to_rad}" upper="${90.0 * deg_to_rad}" effort="${wrist_2_max_effort}" velocity="${wrist_2_max_vel}" />
+      <limit lower="${-wrist_6_range * deg_to_rad}" upper="${wrist_6_range * deg_to_rad}" effort="${wrist_2_max_effort}" velocity="${wrist_2_max_vel}" />
       <dynamics friction="${wrist_friction}" damping="${wrist_damping}"/>
       <safety_controller k_position="20"
                          k_velocity="20"
-                         soft_lower_limit="${-90.0 * deg_to_rad + wrist_eps}"
-                         soft_upper_limit="${ 90.0 * deg_to_rad - wrist_eps}" />
+                         soft_lower_limit="${-wrist_6_range * deg_to_rad + wrist_eps}"
+                         soft_upper_limit="${ wrist_6_range * deg_to_rad - wrist_eps}" />
     </joint>
     <link name="${name}_${side}_7_link">
