Commit message: Add robot urdf file for tf and hey5. Modified ftsensor urdf

File: reemc_description/robots/reemc_full_ft_hey5.urdf.xacro (robot description, xacro)
@@ -40,5 +40,6 @@
   <xacro:include filename="$(find reemc_description)/urdf/arm/arm.urdf.xacro" />
   <!-- Hand -->
-  <xacro:include filename="$(find reemc_description)/urdf/hand/hand.urdf.xacro" />
+<!--  <xacro:include filename="$(find reemc_description)/urdf/hand/hand.urdf.xacro" /> -->
+  <xacro:include filename="$(find hey5_description)/urdf/hey5_hand.urdf.xacro" />
   <!-- Sensors -->
   <xacro:include filename="$(find reemc_description)/urdf/sensors/imu.urdf.xacro" />
@@ -46,4 +47,5 @@
   <xacro:include filename="$(find reemc_description)/urdf/sensors/stereo_camera.urdf.xacro" />
   <xacro:include filename="$(find reemc_description)/urdf/sensors/back_camera.urdf.xacro" />
+  <xacro:include filename="$(find reemc_description)/urdf/sensors/ftsensor.urdf.xacro" />
   <!-- Generic simulator_gazebo plugins -->
   <xacro:include filename="$(find reemc_description)/gazebo/gazebo.urdf.xacro" />
@@ -58,6 +60,16 @@
   <xacro:reem_arm name="arm" parent="torso_2_link" side="right" reflect="1.0"  />
   <xacro:reem_arm name="arm" parent="torso_2_link" side="left"  reflect="-1.0" />
-  <xacro:reem_hand name="hand" parent="arm_right_tool_link" side="right" reflect="1.0"  />
-  <xacro:reem_hand name="hand" parent="arm_left_tool_link"  side="left"  reflect="-1.0" />
+  <xacro:ft_sensor name="wrist" parent="arm_right_tool_link" side="right" reflect="1.0"  />
+  <xacro:ft_sensor name="wrist" parent="arm_left_tool_link"  side="left"  reflect="-1.0" />
+<!--
+  <xacro:reem_hand name="hand" parent="wrist_right_ft_tool_link" side="right" reflect="1.0"  />
+  <xacro:reem_hand name="hand" parent="wrist_left_ft_tool_link"  side="left"  reflect="-1.0" />
+-->
+  <xacro:hey5_hand parent="wrist_right_ft_tool_link" name="hand_right" reflect="1" >
+    <origin xyz="0 0 0" rpy="0 0 0" />
+  </xacro:hey5_hand>
+  <xacro:hey5_hand parent="wrist_left_ft_tool_link" name="hand_left" reflect="-1" >
+    <origin xyz="0 0 0" rpy="${180 * deg_to_rad} 0 0" />
+  </xacro:hey5_hand>
   <!-- stereo camera -->
   <!-- IMPORTANT: focal_length = image_width/(2tan(hfov/2)) -->

File: reemc_description/urdf/sensors/ftsensor.urdf.xacro (robot description, xacro)
@@ -37,5 +37,5 @@
     </joint>
     <!--***********************-->
-    <!--        TOOL           -->
+    <!--       FT TOOL           -->
     <!--***********************-->
     <link name="${name}_${side}_ft_tool_link">
@@ -45,14 +45,14 @@
       </inertial>
       <visual>
-        <origin xyz="0.001 0 0" rpy="0 0 0" />
+        <origin xyz="0.0 0 0" rpy="0 ${90.0 * deg_to_rad} 0" />
         <geometry>
-          <cylinder radius="0.005" length="0.005"/>
+          <cylinder radius="${0.05*0.5}" length="0.00975"/>
         </geometry>
         <material name="FlatBlack" />
       </visual>
       <collision>
-        <origin xyz="0.001 0 0" rpy="0 0 0" />
+        <origin xyz="0.0 0 0" rpy="0 ${90.0 * deg_to_rad} 0" />
         <geometry>
-          <cylinder radius="0.005" length="0.005"/>
+          <cylinder radius="${0.05*0.5}" length="0.00975"/>
         </geometry>
       </collision>
@@ -61,6 +61,5 @@
       <parent link="${name}_${side}_ft_link" />
       <child link="${name}_${side}_ft_tool_link" />
-      <!--<origin xyz="0 0 ${0.0157*0.5}" rpy="0 0 0" />-->
-      <origin xyz="0 0 ${0.0157*0.5}" rpy="${-90.0 * deg_to_rad} ${-90.0 * deg_to_rad} 0" />
+      <origin xyz="0 0 ${0.0157*0.5 + 0.00975*0.5}" rpy="${-90.0 * deg_to_rad} ${-90.0 * deg_to_rad} 0" />
     </joint>
 </xacro:macro>

Commit message: Remove comments

File: reemc_description/robots/reemc_full_ft_hey5.urdf.xacro (robot description, xacro)
@@ -39,6 +39,5 @@
   <!-- Arm -->
   <xacro:include filename="$(find reemc_description)/urdf/arm/arm.urdf.xacro" />
-  <!-- Hand -->
-<!--  <xacro:include filename="$(find reemc_description)/urdf/hand/hand.urdf.xacro" /> -->
+  <!-- Hey5 Hand -->
   <xacro:include filename="$(find hey5_description)/urdf/hey5_hand.urdf.xacro" />
   <!-- Sensors -->
@@ -62,8 +61,4 @@
   <xacro:ft_sensor name="wrist" parent="arm_right_tool_link" side="right" reflect="1.0"  />
   <xacro:ft_sensor name="wrist" parent="arm_left_tool_link"  side="left"  reflect="-1.0" />
-<!--
-  <xacro:reem_hand name="hand" parent="wrist_right_ft_tool_link" side="right" reflect="1.0"  />
-  <xacro:reem_hand name="hand" parent="wrist_left_ft_tool_link"  side="left"  reflect="-1.0" />
--->
   <xacro:hey5_hand parent="wrist_right_ft_tool_link" name="hand_right" reflect="1" >
     <origin xyz="0 0 0" rpy="0 0 0" />

File: reemc_description/urdf/hand/hand.urdf.xacro (robot description, xacro)
@@ -147,5 +147,4 @@
       <parent link="${parent}" />
       <child link="${name}_${side}_palm_link" />
-<!--      <origin xyz="0 0 0" rpy="${-90.0 * deg_to_rad} ${-90.0 * deg_to_rad} 0" /> -->
       <origin xyz="0 0 0" rpy="0 0 0" />
     </joint>

Commit message: Add realsense camera

File: reemc_description/robots/reemc_full_ft_hey5.urdf.xacro (robot description, xacro)
@@ -11,4 +11,9 @@
         xmlns:controller="http://playerstage.sourceforge.net/gazebo/xmlschema/#controller"
         xmlns:interface="http://playerstage.sourceforge.net/gazebo/xmlschema/#interface">
+  <xacro:arg name="head_version" default="v1"/>
+  <xacro:property name="head_version" value="$(arg head_version)" />
+  <xacro:if value="${head_version not in ['v0','v1']}">
+    <xacro:wrong_head_version/>
+  </xacro:if>
   <link name="base_link">
     <inertial>
@@ -36,5 +41,5 @@
   <xacro:include filename="$(find reemc_description)/urdf/torso/torso.urdf.xacro" />
   <!-- Head -->
-  <xacro:include filename="$(find reemc_description)/urdf/head/head.urdf.xacro" />
+  <xacro:include filename="$(find reemc_description)/urdf/head/head_${head_version}.urdf.xacro" />
   <!-- Arm -->
   <xacro:include filename="$(find reemc_description)/urdf/arm/arm.urdf.xacro" />
@@ -44,5 +49,4 @@
   <xacro:include filename="$(find reemc_description)/urdf/sensors/imu.urdf.xacro" />
   <xacro:include filename="$(find reemc_description)/urdf/sensors/laser.urdf.xacro" />
-  <xacro:include filename="$(find reemc_description)/urdf/sensors/stereo_camera.urdf.xacro" />
   <xacro:include filename="$(find reemc_description)/urdf/sensors/back_camera.urdf.xacro" />
   <xacro:include filename="$(find reemc_description)/urdf/sensors/ftsensor.urdf.xacro" />
@@ -51,4 +55,19 @@
   <!-- Materials for visualization -->
   <xacro:include filename="$(find reemc_description)/urdf/materials.urdf.xacro" />
+  <xacro:if value="${head_version == 'v0'}">
+    <!-- stereo camera -->
+    <!-- IMPORTANT: focal_length = image_width/(2tan(hfov/2)) -->
+    <xacro:include filename="$(find reemc_description)/urdf/sensors/stereo_camera.urdf.xacro" />
+    <xacro:reemc_stereo_camera parent="head_2_link" name="stereo" focal_length="461.943804" hfov="${71.0*deg_to_rad}" image_format="B8G8R8" image_width="659" image_height="493">
+    <!-- The following transformations expresses the pose of the stereo_link (X pointing forward, Z upwards and Y leftwards, contrary to the stereo_optical_link which has Z pointing forward) wrt  head_2_link. -->
+      <origin xyz="0.08203  -0.0935  0.0365" rpy="1.56293 -0.00855922 -0.0201307" />
+    </xacro:reemc_stereo_camera>
+  </xacro:if>
+  <xacro:if value="${head_version == 'v1'}">
+    <xacro:include filename="$(find realsense_gazebo_plugin)/urdf/d435.urdf.xacro" />
+      <sensor_d435 parent="head_2_link">
+        <origin xyz="0.018894 -0.187954 0" rpy="${90.0*deg_to_rad} 0 0"/>
+      </sensor_d435>
+  </xacro:if>
   <!-- Now we can start using the macros included above to define the actual robot -->
   <!-- The reflect parameter takes the value 1 or -1 to respectively distinguish right from left side in expressions -->
@@ -67,10 +86,4 @@
     <origin xyz="0 0 0" rpy="${180 * deg_to_rad} 0 0" />
   </xacro:hey5_hand>
-  <!-- stereo camera -->
-  <!-- IMPORTANT: focal_length = image_width/(2tan(hfov/2)) -->
-  <xacro:reemc_stereo_camera parent="head_2_link" name="stereo" focal_length="461.943804" hfov="${71.0*deg_to_rad}" image_format="B8G8R8" image_width="659" image_height="493">
-<!-- The following transformations expresses the pose of the stereo_link (X pointing forward, Z upwards and Y leftwards, contrary to the stereo_optical_link which has Z pointing forward) wrt  head_2_link. -->
-    <origin xyz="0.08203  -0.0935  0.0365" rpy="1.56293 -0.00855922 -0.0201307" />
-  </xacro:reemc_stereo_camera>
   <xacro:reemc_back_camera parent="torso_2_link" name="back_camera" focal_length="376.002379" hfov="${89.999451423*deg_to_rad}" image_format="B8G8R8" image_width="752" image_height="480" >
     <!-- The following transformations expresses the pose of the back_camera_link (X pointing forward, Z upwards and Y leftwards, contrary to the stereo_optical_link which has Z pointing forward) wrt  torso_2_link. -->

File: reemc_description/urdf/head/head_v1.urdf.xacro (robot description, xacro)
@@ -23,9 +23,9 @@
     <link name="${name}_link">
       <inertial>
-        <origin xyz="0.01819	0.00248	-0.00517" rpy="0 0 0" />
-        <mass value="1.11967" />
+        <origin xyz="0.014823 -0.000253 -0.008383" rpy="0 0 0" />
+        <mass value="0.646763" />
         <!-- NOTE: Assuming cylinder with r=0.06, h=0.08 -->
 <!--         <inertia ixx="0.0014125"  ixy="0"  ixz="0" iyy="0.0014125" iyz="0" izz="0.0017738" /> -->
-        <inertia ixx="0.00111370229"  ixy="0.00003992198"  ixz="-0.00012464155" iyy="0.00111361487" iyz="0.00001943162" izz="0.00114794061" />
+        <inertia ixx="0.001175"  ixy="-0.000003"  ixz="0.000012" iyy="0.001273" iyz="-0.000008" izz="0.001132" />
       </inertial>
       <visual>
@@ -69,15 +69,15 @@
     <link name="${name}_link">
       <inertial>
-        <origin xyz="0.01183 -0.08098 0.00104" rpy="0 0 0" />
-        <mass value="1.63134" />
+        <origin xyz="-0.023981 -0.100591 0.000294" rpy="0 0 0" />
+        <mass value="0.920999" />
         <!-- NOTE: Assuming box with d=0.28433, w=0.20302, h=0.26741 -->
 <!--         <inertia ixx="0.011353"  ixy="0"  ixz="0" iyy="0.012294" iyz="0" izz="0.015345" /> -->
         <!--NOTE: Low (0.1 or lower) diagonal inertia values make Gazebo 1.0.2 simulation unstable when head sensors are added.-->
-        <inertia ixx="0.00640199093"  ixy="0.00012197067"  ixz="-0.00000897011" iyy="0.00676228591" iyz="-0.0000552329" izz="0.00614192438" />
+        <inertia ixx="0.005972"  ixy="-0.000046"  ixz="0.000006" iyy="0.006327" iyz="0.000030" izz="0.006213" />
       </inertial>
       <visual>
-        <origin rpy="0 0 0" xyz="-0.03 0 0"/> <!--TODO: Remove offset when good meshes arrive-->
+        <origin rpy="0 0 0" xyz="0 0 0"/>
         <geometry>
-          <mesh filename="package://reemc_description/meshes/head/head_2.dae" />
+          <mesh filename="package://reemc_description/meshes/head/head_2_v1.stl" />
         </geometry>
         <material name="LightGrey" />
@@ -93,5 +93,5 @@
       <parent link="${parent}"/>
         <child link="${name}_link"/>
-      <origin xyz="0.0445 0 0" rpy="${-90.0 * deg_to_rad} 0 0" />
+      <origin xyz="0.0445 0 0" rpy="${-90.0 * deg_to_rad} ${0.0 * deg_to_rad}  0" />
       <axis xyz="0 0 1" />
       <limit lower="${-15.0 * deg_to_rad}" upper="${45.0 * deg_to_rad}" effort="3.26" velocity="${head_max_vel}" />
