Commit message: Update the rest of the robot files with the new head version

File: reemc_description/robots/reemc_full_chessboard.urdf.xacro (robot description, xacro)
@@ -11,4 +11,9 @@
         xmlns:controller="http://playerstage.sourceforge.net/gazebo/xmlschema/#controller"
         xmlns:interface="http://playerstage.sourceforge.net/gazebo/xmlschema/#interface">
+  <xacro:arg name="head_version" default="v1"/>
+  <xacro:property name="head_version" value="$(arg head_version)" />
+  <xacro:if value="${head_version not in ['v0','v1']}">
+    <xacro:wrong_head_version/>
+  </xacro:if>
   <link name="base_link">
     <inertial>
@@ -36,5 +41,5 @@
   <xacro:include filename="$(find reemc_description)/urdf/torso/torso.urdf.xacro" />
   <!-- Head -->
-  <xacro:include filename="$(find reemc_description)/urdf/head/head.urdf.xacro" />
+  <xacro:include filename="$(find reemc_description)/urdf/head/head_${head_version}.urdf.xacro" />
   <!-- Arm -->
   <xacro:include filename="$(find reemc_description)/urdf/arm/arm.urdf.xacro" />
@@ -44,5 +49,4 @@
   <xacro:include filename="$(find reemc_description)/urdf/sensors/imu.urdf.xacro" />
   <xacro:include filename="$(find reemc_description)/urdf/sensors/laser.urdf.xacro" />
-  <xacro:include filename="$(find reemc_description)/urdf/sensors/stereo_camera.urdf.xacro" />
   <xacro:include filename="$(find reemc_description)/urdf/sensors/back_camera.urdf.xacro" />
   <xacro:include filename="$(find reemc_description)/urdf/sensors/ftsensor.urdf.xacro" />
@@ -51,4 +55,19 @@
   <!-- Materials for visualization -->
   <xacro:include filename="$(find reemc_description)/urdf/materials.urdf.xacro" />
+  <xacro:if value="${head_version == 'v0'}">
+    <!-- stereo camera -->
+    <!-- IMPORTANT: focal_length = image_width/(2tan(hfov/2)) -->
+    <xacro:include filename="$(find reemc_description)/urdf/sensors/stereo_camera.urdf.xacro" />
+    <xacro:reemc_stereo_camera parent="head_2_link" name="stereo" focal_length="461.943804" hfov="${71.0*deg_to_rad}" image_format="B8G8R8" image_width="659" image_height="493">
+    <!-- The following transformations expresses the pose of the stereo_link (X pointing forward, Z upwards and Y leftwards, contrary to the stereo_optical_link which has Z pointing forward) wrt  head_2_link. -->
+      <origin xyz="0.08203  -0.0935  0.0365" rpy="1.56293 -0.00855922 -0.0201307" />
+    </xacro:reemc_stereo_camera>
+  </xacro:if>
+  <xacro:if value="${head_version == 'v1'}">
+    <xacro:include filename="$(find realsense_gazebo_plugin)/urdf/d435.urdf.xacro" />
+      <sensor_d435 parent="head_2_link">
+        <origin xyz="0.018894 -0.187954 0" rpy="${90.0*deg_to_rad} 0 0"/>
+      </sensor_d435>
+  </xacro:if>
   <!-- Now we can start using the macros included above to define the actual robot -->
   <!-- The reflect parameter takes the value 1 or -1 to respectively distinguish right from left side in expressions -->
@@ -61,10 +80,4 @@
   <xacro:ft_sensor name="wrist" parent="arm_right_tool_link" side="right" reflect="1.0"  />
   <xacro:ft_sensor name="wrist" parent="arm_left_tool_link"  side="left"  reflect="-1.0" />
-  <!-- stereo camera -->
-  <!-- IMPORTANT: focal_length = image_width/(2tan(hfov/2)) -->
-  <xacro:reemc_stereo_camera parent="head_2_link" name="stereo" focal_length="461.943804" hfov="${71.0*deg_to_rad}" image_format="B8G8R8" image_width="659" image_height="493">
-<!-- The following transformations expresses the pose of the stereo_link (X pointing forward, Z upwards and Y leftwards, contrary to the stereo_optical_link which has Z pointing forward) wrt  head_2_link. -->
-    <origin xyz="0.08203  -0.0935  0.0365" rpy="1.56293 -0.00855922 -0.0201307" />
-  </xacro:reemc_stereo_camera>
   <xacro:reemc_back_camera parent="torso_2_link" name="back_camera" focal_length="376.002379" hfov="${89.999451423*deg_to_rad}" image_format="B8G8R8" image_width="752" image_height="480" >
     <!-- The following transformations expresses the pose of the back_camera_link (X pointing forward, Z upwards and Y leftwards, contrary to the stereo_optical_link which has Z pointing forward) wrt  torso_2_link. -->

File: reemc_description/robots/reemc_full_no_hands.urdf.xacro (robot description, xacro)
@@ -11,4 +11,9 @@
         xmlns:controller="http://playerstage.sourceforge.net/gazebo/xmlschema/#controller"
         xmlns:interface="http://playerstage.sourceforge.net/gazebo/xmlschema/#interface">
+  <xacro:arg name="head_version" default="v1"/>
+  <xacro:property name="head_version" value="$(arg head_version)" />
+  <xacro:if value="${head_version not in ['v0','v1']}">
+    <xacro:wrong_head_version/>
+  </xacro:if>
   <link name="base_link">
     <inertial>
@@ -36,5 +41,5 @@
   <xacro:include filename="$(find reemc_description)/urdf/torso/torso.urdf.xacro" />
   <!-- Head -->
-  <xacro:include filename="$(find reemc_description)/urdf/head/head.urdf.xacro" />
+  <xacro:include filename="$(find reemc_description)/urdf/head/head_${head_version}.urdf.xacro" />
   <!-- Arm -->
   <xacro:include filename="$(find reemc_description)/urdf/arm/arm.urdf.xacro" />
@@ -44,5 +49,4 @@
   <xacro:include filename="$(find reemc_description)/urdf/sensors/imu.urdf.xacro" />
   <xacro:include filename="$(find reemc_description)/urdf/sensors/laser.urdf.xacro" />
-  <xacro:include filename="$(find reemc_description)/urdf/sensors/stereo_camera.urdf.xacro" />
   <xacro:include filename="$(find reemc_description)/urdf/sensors/back_camera.urdf.xacro" />
   <xacro:include filename="$(find reemc_description)/urdf/sensors/ftsensor.urdf.xacro" />
@@ -51,4 +55,19 @@
   <!-- Materials for visualization -->
   <xacro:include filename="$(find reemc_description)/urdf/materials.urdf.xacro" />
+  <xacro:if value="${head_version == 'v0'}">
+    <!-- stereo camera -->
+    <!-- IMPORTANT: focal_length = image_width/(2tan(hfov/2)) -->
+    <xacro:include filename="$(find reemc_description)/urdf/sensors/stereo_camera.urdf.xacro" />
+    <xacro:reemc_stereo_camera parent="head_2_link" name="stereo" focal_length="461.943804" hfov="${71.0*deg_to_rad}" image_format="B8G8R8" image_width="659" image_height="493">
+    <!-- The following transformations expresses the pose of the stereo_link (X pointing forward, Z upwards and Y leftwards, contrary to the stereo_optical_link which has Z pointing forward) wrt  head_2_link. -->
+      <origin xyz="0.08203  -0.0935  0.0365" rpy="1.56293 -0.00855922 -0.0201307" />
+    </xacro:reemc_stereo_camera>
+  </xacro:if>
+  <xacro:if value="${head_version == 'v1'}">
+    <xacro:include filename="$(find realsense_gazebo_plugin)/urdf/d435.urdf.xacro" />
+      <sensor_d435 parent="head_2_link">
+        <origin xyz="0.018894 -0.187954 0" rpy="${90.0*deg_to_rad} 0 0"/>
+      </sensor_d435>
+  </xacro:if>
   <!-- Now we can start using the macros included above to define the actual robot -->
   <!-- The reflect parameter takes the value 1 or -1 to respectively distinguish right from left side in expressions -->
@@ -61,10 +80,4 @@
   <xacro:ft_sensor name="wrist" parent="arm_right_tool_link" side="right" reflect="1.0"  />
   <xacro:ft_sensor name="wrist" parent="arm_left_tool_link"  side="left"  reflect="-1.0" />
-  <!-- stereo camera -->
-  <!-- IMPORTANT: focal_length = image_width/(2tan(hfov/2)) -->
-  <xacro:reemc_stereo_camera parent="head_2_link" name="stereo" focal_length="461.943804" hfov="${71.0*deg_to_rad}" image_format="B8G8R8" image_width="659" image_height="493">
-<!-- The following transformations expresses the pose of the stereo_link (X pointing forward, Z upwards and Y leftwards, contrary to the stereo_optical_link which has Z pointing forward) wrt  head_2_link. -->
-    <origin xyz="0.08203  -0.0935  0.0365" rpy="1.56293 -0.00855922 -0.0201307" />
-  </xacro:reemc_stereo_camera>
   <xacro:reemc_back_camera parent="torso_2_link" name="back_camera" focal_length="376.002379" hfov="${89.999451423*deg_to_rad}" image_format="B8G8R8" image_width="752" image_height="480" >
     <!-- The following transformations expresses the pose of the back_camera_link (X pointing forward, Z upwards and Y leftwards, contrary to the stereo_optical_link which has Z pointing forward) wrt  torso_2_link. -->

File: reemc_description/robots/reemc_lower_body.urdf.xacro (robot description, xacro)
@@ -11,5 +11,10 @@
         xmlns:controller="http://playerstage.sourceforge.net/gazebo/xmlschema/#controller"
         xmlns:interface="http://playerstage.sourceforge.net/gazebo/xmlschema/#interface">
-   <link name="base_link">
+  <xacro:arg name="head_version" default="v1"/>
+  <xacro:property name="head_version" value="$(arg head_version)" />
+  <xacro:if value="${head_version not in ['v0','v1']}">
+    <xacro:wrong_head_version/>
+  </xacro:if>
+  <link name="base_link">
     <inertial>
       <mass value="36.85"/>
@@ -40,5 +45,5 @@
   <xacro:include filename="$(find reemc_description)/urdf/torso/torso.urdf.xacro" />
   <!-- Head -->
-  <xacro:include filename="$(find reemc_description)/urdf/head/head.urdf.xacro" />
+  <xacro:include filename="$(find reemc_description)/urdf/head/head_${head_version}.urdf.xacro" />
   <!-- Arm -->
   <xacro:include filename="$(find reemc_description)/urdf/arm/arm.urdf.xacro" />
@@ -48,5 +53,4 @@
   <xacro:include filename="$(find reemc_description)/urdf/sensors/imu.urdf.xacro" />
   <xacro:include filename="$(find reemc_description)/urdf/sensors/laser.urdf.xacro" />
-  <xacro:include filename="$(find reemc_description)/urdf/sensors/stereo_camera.urdf.xacro" />
   <xacro:include filename="$(find reemc_description)/urdf/sensors/back_camera.urdf.xacro" />
   <!-- Generic simulator_gazebo plugins -->
@@ -54,4 +58,19 @@
   <!-- Materials for visualization -->
   <xacro:include filename="$(find reemc_description)/urdf/materials.urdf.xacro" />
+  <xacro:if value="${head_version == 'v0'}">
+    <!-- stereo camera -->
+    <!-- IMPORTANT: focal_length = image_width/(2tan(hfov/2)) -->
+    <xacro:include filename="$(find reemc_description)/urdf/sensors/stereo_camera.urdf.xacro" />
+    <xacro:reemc_stereo_camera parent="head_2_link" name="stereo" focal_length="461.943804" hfov="${71.0*deg_to_rad}" image_format="B8G8R8" image_width="659" image_height="493">
+    <!-- The following transformations expresses the pose of the stereo_link (X pointing forward, Z upwards and Y leftwards, contrary to the stereo_optical_link which has Z pointing forward) wrt  head_2_link. -->
+      <origin xyz="0.08203  -0.0935  0.0365" rpy="1.56293 -0.00855922 -0.0201307" />
+    </xacro:reemc_stereo_camera>
+  </xacro:if>
+  <xacro:if value="${head_version == 'v1'}">
+    <xacro:include filename="$(find realsense_gazebo_plugin)/urdf/d435.urdf.xacro" />
+      <sensor_d435 parent="head_2_link">
+        <origin xyz="0.018894 -0.187954 0" rpy="${90.0*deg_to_rad} 0 0"/>
+      </sensor_d435>
+  </xacro:if>
   <!-- Now we can start using the macros included above to define the actual robot -->
   <!-- The reflect parameter takes the value 1 or -1 to respectively distinguish right from left side in expressions -->

Commit message: Add generic camera frame

File: reemc_description/robots/reemc_full_chessboard.urdf.xacro (robot description, xacro)
@@ -12,4 +12,5 @@
         xmlns:interface="http://playerstage.sourceforge.net/gazebo/xmlschema/#interface">
   <xacro:arg name="head_version" default="v1"/>
+  <xacro:property name="camera" value="${'camera_color' if head_version == 'v1' else 'stereo'}"/>
   <xacro:property name="head_version" value="$(arg head_version)" />
   <xacro:if value="${head_version not in ['v0','v1']}">
@@ -70,4 +71,18 @@
       </sensor_d435>
   </xacro:if>
+  <joint name="camera_optical_frame_joint" type="fixed">
+    <origin xyz="0 0 0" rpy="0 0 0" />
+    <parent link="${camera}_optical_frame"/>
+    <child link="camera_optical_frame"/>
+  </joint>
+    <!-- optical frame for the stereo camera, with z-forward notation, this is the frame stereo camera images users should refer to -->
+  <link name="camera_optical_frame" type="camera">
+    <inertial>
+      <mass value="0.01" />
+      <origin xyz="0 0 0" rpy="0 0 0" />
+      <inertia ixx="0"  ixy="0"  ixz="0"
+               iyy="0"  iyz="0"  izz="0" />
+    </inertial>
+  </link>
   <!-- Now we can start using the macros included above to define the actual robot -->
   <!-- The reflect parameter takes the value 1 or -1 to respectively distinguish right from left side in expressions -->

File: reemc_description/robots/reemc_full_ft_hey5.urdf.xacro (robot description, xacro)
@@ -12,4 +12,5 @@
         xmlns:interface="http://playerstage.sourceforge.net/gazebo/xmlschema/#interface">
   <xacro:arg name="head_version" default="v1"/>
+  <xacro:property name="camera" value="${'camera_color' if head_version == 'v1' else 'stereo'}"/>
   <xacro:property name="head_version" value="$(arg head_version)" />
   <xacro:if value="${head_version not in ['v0','v1']}">
@@ -70,4 +71,18 @@
       </sensor_d435>
   </xacro:if>
+  <joint name="camera_optical_frame_joint" type="fixed">
+  	<origin xyz="0 0 0" rpy="0 0 0" />
+    <parent link="${camera}_optical_frame"/>
+    <child link="camera_optical_frame"/>
+  </joint>
+    <!-- optical frame for the stereo camera, with z-forward notation, this is the frame stereo camera images users should refer to -->
+  <link name="camera_optical_frame" type="camera">
+    <inertial>
+      <mass value="0.01" />
+      <origin xyz="0 0 0" rpy="0 0 0" />
+      <inertia ixx="0"  ixy="0"  ixz="0"
+               iyy="0"  iyz="0"  izz="0" />
+    </inertial>
+  </link>
   <!-- Now we can start using the macros included above to define the actual robot -->
   <!-- The reflect parameter takes the value 1 or -1 to respectively distinguish right from left side in expressions -->

File: reemc_description/robots/reemc_full_no_hands.urdf.xacro (robot description, xacro)
@@ -12,4 +12,5 @@
         xmlns:interface="http://playerstage.sourceforge.net/gazebo/xmlschema/#interface">
   <xacro:arg name="head_version" default="v1"/>
+  <xacro:property name="camera" value="${'camera_color' if head_version == 'v1' else 'stereo'}"/>
   <xacro:property name="head_version" value="$(arg head_version)" />
   <xacro:if value="${head_version not in ['v0','v1']}">
@@ -70,4 +71,18 @@
       </sensor_d435>
   </xacro:if>
+  <joint name="camera_optical_frame_joint" type="fixed">
+    <origin xyz="0 0 0" rpy="0 0 0" />
+    <parent link="${camera}_optical_frame"/>
+    <child link="camera_optical_frame"/>
+  </joint>
+    <!-- optical frame for the stereo camera, with z-forward notation, this is the frame stereo camera images users should refer to -->
+  <link name="camera_optical_frame" type="camera">
+    <inertial>
+      <mass value="0.01" />
+      <origin xyz="0 0 0" rpy="0 0 0" />
+      <inertia ixx="0"  ixy="0"  ixz="0"
+               iyy="0"  iyz="0"  izz="0" />
+    </inertial>
+  </link>
   <!-- Now we can start using the macros included above to define the actual robot -->
   <!-- The reflect parameter takes the value 1 or -1 to respectively distinguish right from left side in expressions -->

File: reemc_description/robots/reemc_lower_body.urdf.xacro (robot description, xacro)
@@ -12,4 +12,5 @@
         xmlns:interface="http://playerstage.sourceforge.net/gazebo/xmlschema/#interface">
   <xacro:arg name="head_version" default="v1"/>
+  <xacro:property name="camera" value="${'camera_color' if head_version == 'v1' else 'stereo'}"/>
   <xacro:property name="head_version" value="$(arg head_version)" />
   <xacro:if value="${head_version not in ['v0','v1']}">
@@ -73,4 +74,18 @@
       </sensor_d435>
   </xacro:if>
+  <joint name="camera_optical_frame_joint" type="fixed">
+    <origin xyz="0 0 0" rpy="0 0 0" />
+    <parent link="${camera}_optical_frame"/>
+    <child link="camera_optical_frame"/>
+  </joint>
+    <!-- optical frame for the stereo camera, with z-forward notation, this is the frame stereo camera images users should refer to -->
+  <link name="camera_optical_frame" type="camera">
+    <inertial>
+      <mass value="0.01" />
+      <origin xyz="0 0 0" rpy="0 0 0" />
+      <inertia ixx="0"  ixy="0"  ixz="0"
+               iyy="0"  iyz="0"  izz="0" />
+    </inertial>
+  </link>
   <!-- Now we can start using the macros included above to define the actual robot -->
   <!-- The reflect parameter takes the value 1 or -1 to respectively distinguish right from left side in expressions -->

Commit message: Adding legs v0,v1 specs and setting default version for leg and head to v0 for back-compatibility

File: reemc_description/robots/reemc_full_chessboard.urdf.xacro (robot description, xacro)
@@ -11,5 +11,5 @@
         xmlns:controller="http://playerstage.sourceforge.net/gazebo/xmlschema/#controller"
         xmlns:interface="http://playerstage.sourceforge.net/gazebo/xmlschema/#interface">
-  <xacro:arg name="head_version" default="v1"/>
+  <xacro:arg name="head_version" default="v0"/>
   <xacro:property name="camera" value="${'camera_color' if head_version == 'v1' else 'stereo'}"/>
   <xacro:property name="head_version" value="$(arg head_version)" />

File: reemc_description/robots/reemc_full_ft_hey5.urdf.xacro (robot description, xacro)
@@ -11,5 +11,5 @@
         xmlns:controller="http://playerstage.sourceforge.net/gazebo/xmlschema/#controller"
         xmlns:interface="http://playerstage.sourceforge.net/gazebo/xmlschema/#interface">
-  <xacro:arg name="head_version" default="v1"/>
+  <xacro:arg name="head_version" default="v0"/>
   <xacro:property name="camera" value="${'camera_color' if head_version == 'v1' else 'stereo'}"/>
   <xacro:property name="head_version" value="$(arg head_version)" />

File: reemc_description/robots/reemc_full_no_hands.urdf.xacro (robot description, xacro)
@@ -11,5 +11,5 @@
         xmlns:controller="http://playerstage.sourceforge.net/gazebo/xmlschema/#controller"
         xmlns:interface="http://playerstage.sourceforge.net/gazebo/xmlschema/#interface">
-  <xacro:arg name="head_version" default="v1"/>
+  <xacro:arg name="head_version" default="v0"/>
   <xacro:property name="camera" value="${'camera_color' if head_version == 'v1' else 'stereo'}"/>
   <xacro:property name="head_version" value="$(arg head_version)" />

File: reemc_description/robots/reemc_lower_body.urdf.xacro (robot description, xacro)
@@ -11,5 +11,5 @@
         xmlns:controller="http://playerstage.sourceforge.net/gazebo/xmlschema/#controller"
         xmlns:interface="http://playerstage.sourceforge.net/gazebo/xmlschema/#interface">
-  <xacro:arg name="head_version" default="v1"/>
+  <xacro:arg name="head_version" default="v0"/>
   <xacro:property name="camera" value="${'camera_color' if head_version == 'v1' else 'stereo'}"/>
   <xacro:property name="head_version" value="$(arg head_version)" />

File: reemc_description/urdf/leg/leg.urdf.xacro (robot description, xacro)
@@ -13,4 +13,10 @@
   <xacro:include filename="$(find reemc_description)/urdf/sensors/ftsensor.gazebo.xacro"/>
   <xacro:include filename="$(find reemc_description)/urdf/sensors/laser.urdf.xacro"/>
+  <xacro:arg name="leg_version" default="v0"/>
+  <xacro:property name="leg_version" value="$(arg leg_version)" />
+  <xacro:if value="${leg_version not in ['v0','v1']}">
+    <xacro:wrong_leg_version/>
+  </xacro:if>
+  <xacro:property name="camera" value="${'camera_color' if head_version == 'v1' else 'stereo'}"/>
   <!--Constant parameters-->
   <xacro:property name="leg_friction"       value="1.0" />
@@ -18,16 +24,16 @@
   <xacro:property name="leg_reduction"      value="1.0" />
   <xacro:property name="leg_eps"            value="0.0" />
-  <xacro:property name="leg_1_joint_max_vel"        value="2.35" />
-  <xacro:property name="leg_2_joint_max_vel"        value="2.27" />
-  <xacro:property name="leg_3_joint_max_vel"        value="3.64" />
-  <xacro:property name="leg_4_joint_max_vel"        value="3.225" />
-  <xacro:property name="leg_5_joint_max_vel"        value="2.44" />
-  <xacro:property name="leg_6_joint_max_vel"        value="2.27" />
-  <xacro:property name="leg_1_joint_effort"        value="42.7" />
-  <xacro:property name="leg_2_joint_effort"        value="64.0" />
-  <xacro:property name="leg_3_joint_effort"        value="55.7" />
-  <xacro:property name="leg_4_joint_effort"        value="138.3" />
-  <xacro:property name="leg_5_joint_effort"        value="80.9" />
-  <xacro:property name="leg_6_joint_effort"        value="64.0" />
+  <xacro:property name="leg_1_joint_max_vel"        value="${2.74 if leg_version=='v1' else 2.35}" />
+  <xacro:property name="leg_2_joint_max_vel"        value="${3.94 if leg_version=='v1' else 2.27}" />
+  <xacro:property name="leg_3_joint_max_vel"        value="${6.0  if leg_version=='v1' else 3.64}" />
+  <xacro:property name="leg_4_joint_max_vel"        value="${4.25 if leg_version=='v1' else 3.225}" />
+  <xacro:property name="leg_5_joint_max_vel"        value="${4.0  if leg_version=='v1' else 2.44}" />
+  <xacro:property name="leg_6_joint_max_vel"        value="${3.94 if leg_version=='v1' else 2.27}" />
+  <xacro:property name="leg_1_joint_effort"        value="${50.69 if leg_version=='v1' else 42.7}" />
+  <xacro:property name="leg_2_joint_effort"        value="${71.4  if leg_version=='v1' else 64.0}" />
+  <xacro:property name="leg_3_joint_effort"        value="${62.9  if leg_version=='v1' else 55.7}" />
+  <xacro:property name="leg_4_joint_effort"        value="${140.4 if leg_version=='v1' else 138.3}" />
+  <xacro:property name="leg_5_joint_effort"        value="${91.6  if leg_version=='v1' else 80.9}" />
+  <xacro:property name="leg_6_joint_effort"        value="${71.48 if leg_version=='v1' else 64.0}" />
   <xacro:macro name="reemc_leg" params="name parent side reflect">
     <link name="leg_${side}_1_link">
