Commit message: fixed the transform to the realsense D435 link

File: reemc_description/robots/reemc_full_chessboard.urdf.xacro (robot description, xacro)
@@ -68,5 +68,5 @@
     <xacro:include filename="$(find realsense2_description)/urdf/_d435.urdf.xacro" />
       <sensor_d435 parent="head_2_link" use_nominal_extrinsics="true">
-        <origin xyz="0.018894 -0.187954 0" rpy="${90.0*deg_to_rad} 0 0"/>
+        <origin xyz="0.05175 -0.1632503 0" rpy="${90.0*deg_to_rad} 0 0"/>
       </sensor_d435>
   </xacro:if>

File: reemc_description/robots/reemc_full_ft_hey5.urdf.xacro (robot description, xacro)
@@ -68,5 +68,5 @@
     <xacro:include filename="$(find realsense2_description)/urdf/_d435.urdf.xacro" />
       <sensor_d435 parent="head_2_link" use_nominal_extrinsics="true">
-        <origin xyz="0.018894 -0.187954 0" rpy="${90.0*deg_to_rad} 0 0"/>
+        <origin xyz="0.05175 -0.1632503 0" rpy="${90.0*deg_to_rad} 0 0"/>
       </sensor_d435>
   </xacro:if>

File: reemc_description/robots/reemc_full_no_hands.urdf.xacro (robot description, xacro)
@@ -68,5 +68,5 @@
     <xacro:include filename="$(find realsense2_description)/urdf/_d435.urdf.xacro" />
       <sensor_d435 parent="head_2_link" use_nominal_extrinsics="true">
-        <origin xyz="0.018894 -0.187954 0" rpy="${90.0*deg_to_rad} 0 0"/>
+        <origin xyz="0.05175 -0.1632503 0" rpy="${90.0*deg_to_rad} 0 0"/>
       </sensor_d435>
   </xacro:if>

File: reemc_description/robots/reemc_lower_body.urdf.xacro (robot description, xacro)
@@ -71,5 +71,5 @@
     <xacro:include filename="$(find realsense2_description)/urdf/_d435.urdf.xacro" />
       <sensor_d435 parent="head_2_link" use_nominal_extrinsics="true">
-        <origin xyz="0.018894 -0.187954 0" rpy="${90.0*deg_to_rad} 0 0"/>
+        <origin xyz="0.05175 -0.1632503 0" rpy="${90.0*deg_to_rad} 0 0"/>
       </sensor_d435>
   </xacro:if>
