Commit message: Use custom head transmission.
Tilt joint position limits depend on actual pan joint position.

Refs #9907.

File: reemc_description/urdf/head/head.transmission.xacro (robot description, xacro)
@@ -8,11 +8,61 @@
 -->
 <robot xmlns:xacro="http://ros.org/wiki/xacro">
-  <xacro:macro name="head_transmission" params="name reduction">
-    <transmission name="${name}_trans">
-      <type>transmission_interface/SimpleTransmission</type>
-      <actuator name="${name}_motor" >
-        <mechanicalReduction>${reduction}</mechanicalReduction>
+  <xacro:macro name="head_transmission" params="name">
+    <transmission name="${name}">
+      <type>pal_transmissions/HeadTransmission</type>
+      <actuator name="head_1_motor">
+        <role>independent</role>
+        <mechanicalReduction>1.0</mechanicalReduction>
       </actuator>
-      <joint name="${name}_joint" >
+      <actuator name="head_2_motor">
+        <role>dependent</role>
+        <mechanicalReduction>1.0</mechanicalReduction>
+      </actuator>
+      <joint name="head_1_joint">
+        <role>independent</role>
+        <hardwareInterface>hardware_interface/PositionJointInterface</hardwareInterface>
+      </joint>
+      <joint name="head_2_joint">
+        <role>dependent</role>
+        <limits>
+          <key> ${-50.0 * deg_to_rad} </key>
+          <max> ${ 14.0 * deg_to_rad} </max>
+        </limits>
+        <limits>
+          <key> ${-40.0 * deg_to_rad} </key>
+          <max> ${ 18.0 * deg_to_rad} </max>
+        </limits>
+        <limits>
+          <key> ${-30.0 * deg_to_rad} </key>
+          <max> ${ 27.0 * deg_to_rad} </max>
+        </limits>
+        <limits>
+          <key> ${-20.0 * deg_to_rad} </key>
+          <max> ${ 39.0 * deg_to_rad} </max>
+        </limits>
+        <limits>
+          <key> ${-10.0 * deg_to_rad} </key>
+          <max> ${ 45.0 * deg_to_rad} </max>
+        </limits>
+        <limits>
+          <key> ${10.0 * deg_to_rad} </key>
+          <max> ${45.0 * deg_to_rad} </max>
+        </limits>
+        <limits>
+          <key> ${20.0 * deg_to_rad} </key>
+          <max> ${39.0 * deg_to_rad} </max>
+        </limits>
+        <limits>
+          <key> ${30.0 * deg_to_rad} </key>
+          <max> ${27.0 * deg_to_rad} </max>
+        </limits>
+        <limits>
+          <key> ${40.0 * deg_to_rad} </key>
+          <max> ${18.0 * deg_to_rad} </max>
+        </limits>
+        <limits>
+          <key> ${50.0 * deg_to_rad} </key>
+          <max> ${14.0 * deg_to_rad} </max>
+        </limits>
         <hardwareInterface>hardware_interface/PositionJointInterface</hardwareInterface>
       </joint>

File: reemc_description/urdf/head/head.urdf.xacro (robot description, xacro)
@@ -62,6 +62,4 @@
        <implicitSpringDamper>1</implicitSpringDamper>
     </gazebo>
-    <!-- extensions -->
-    <xacro:head_transmission name="${name}" reduction="1" />
   </xacro:macro>
   <!--************************-->
@@ -102,5 +100,5 @@
                          k_velocity="20"
                          soft_lower_limit="${-15.0 * deg_to_rad + head_eps}"
-                         soft_upper_limit="${ 20.0 * deg_to_rad}" />
+                         soft_upper_limit="${ 45.0 * deg_to_rad}" />
     </joint>
     <gazebo reference="${name}_link">
@@ -115,10 +113,9 @@
       <origin xyz="0.11 -0.195 0.0" rpy="1.57 0.0 0.0" />
     </xacro:range_reem>
-    <!-- extensions -->
-    <xacro:head_transmission name="${name}" reduction="1" />
   </xacro:macro>
   <xacro:macro name="reem_head" params="name parent">
     <xacro:reem_head_1 name="${name}_1" parent="${parent}" />
     <xacro:reem_head_2 name="${name}_2" parent="${name}_1_link"/>
+    <xacro:head_transmission name="${name}"/>
   </xacro:macro>
 </robot>
