Commit message: Added reemc specifics to walking params, and reverted torso to revolute joint

File: reemc_description/urdf/torso/torso.urdf.xacro (robot description, xacro)
@@ -34,5 +34,5 @@
       </visual>
     </link>
-    <joint name="${name}_1_joint" type="fixed">
+    <joint name="${name}_1_joint" type="revolute">
       <parent link="${parent}"/>
       <child link="${name}_1_link"/>
@@ -70,5 +70,5 @@
       </collision>
     </link>
-    <joint name="${name}_2_joint" type="fixed">
+    <joint name="${name}_2_joint" type="revolute">
       <parent link="${name}_1_link" />
       <child link="${name}_2_link" />
